Commit message: Cleanup readme
Signed-off-by: Yadunund <yadunund@gmail.com>

File: ieec_description/urdf/ur_gz.urdf.xacro (robot description, xacro)
@@ -32,5 +32,5 @@
   <link name="world" />
   <link name="ground_plane">
-    <visual>
+    <!-- <visual>
       <origin rpy="0 0 0" xyz="0 0 0"/>
       <geometry>
@@ -40,5 +40,5 @@
         <color rgba="1 1 1 0.5"/>
       </material>
-    </visual>
+    </visual> -->
     <collision>
       <origin rpy="0 0 0" xyz="0 0 0"/>
