Commit message: change ft sensor attach_joint from fixed to revolute and add preserveFixedJoint to preserve the joint in gazebo

File: aic_assets/models/ATI_Axia80_M20/axia80_m20_macro.xacro (robot description, xacro)
@@ -17,10 +17,8 @@
       </inertial>
     </link>
-    <joint name="${tf_prefix}attach_joint" type="revolute">
+    <joint name="${tf_prefix}attach_joint" type="fixed">
       <origin xyz="0 0 ${adapter_offset}" rpy="0 0 0"/>
       <parent link="${tf_prefix}base_link"/>
       <child link="${tf_prefix}tool_link"/>
-      <axis xyz="0 0 1"/>
-      <limit lower="-0.0001" upper="0.0001" effort="9999" velocity="0.001"/>
     </joint>
     <link name="${tf_prefix}tool_link">
@@ -52,4 +50,5 @@
     </link>
     <gazebo reference="${tf_prefix}attach_joint">
+      <preserveFixedJoint>true</preserveFixedJoint>
       <sensor name="AtiForceTorqueSensor" type="force_torque">
         <always_on>1</always_on>

Commit message: Add and fix contact sensor.

File: aic_assets/models/ATI_Axia80_M20/axia80_m20_macro.xacro (robot description, xacro)
@@ -4,5 +4,5 @@
   <xacro:property name="name" value="axia80_m20"/>
   <!-- TF prefix parameter -->
-  <xacro:property name="tf_prefix" value="ati"/>
+  <xacro:property name="tf_prefix" value="ati/"/>
   <!-- adapter_offset is the effective length that the adapter adds to the endeffector -->
   <xacro:property name="adapter_offset" value="0.0245"/>
@@ -106,13 +106,11 @@
       <sensor name="contact_sensor" type="contact">
         <contact>
-          <collision>collision1</collision>
+          <!-- The reason for the convoluted collision name reference is due to URDF to SDF
+          conversion prepending and appending names to the collision name. The current workaround
+          is provide an exact name -->
+          <collision>${tf_prefix}tool_link_fixed_joint_lump__collision1_collision</collision>
+          <topic>collision/tool_link</topic>
         </contact>
       </sensor>
-      <!-- Reduce contact stiffness and damping for better stability -->
-      <kp>100000</kp>
-      <kd>100</kd>
-      <!-- Reduce friction in order to get smoother simulated force -->
-      <mu1>0.01</mu1>
-      <mu2>0.01</mu2>
     </gazebo>
   </xacro:macro>
