Commit message: add urdf files and update ur_gz

File: aic_assets/models/Axia80 M20/axia80_m20_macro.xacro (robot description, xacro)
@@ -1,14 +1,12 @@
 <?xml version="1.0" ?>
 <robot xmlns:xacro="http://wiki.ros.org/xacro">
-  <!-- robot name parameter -->
-  <xacro:property name="name" value="axia80_m20"/>
   <!-- TF prefix parameter -->
   <xacro:property name="tf_prefix" value="ati/"/>
   <!-- adapter_offset is the effective length that the adapter adds to the endeffector -->
-  <xacro:property name="adapter_offset" value="0.0245"/>
-  <xacro:macro name="axia80_m20" params="name tf_prefix">
+  <!-- <xacro:property name="adapter_offset" value="0.0245"/> -->
+  <xacro:macro name="axia80_m20" params="tf_prefix">
     <link name="${tf_prefix}base_link">
       <inertial>
-        <origin xyz="0 0 ${adapter_offset / 2}" rpy="0 0 0"/>
+        <origin xyz="0 0 0" rpy="0 0 0"/>
         <mass value="0.36"/>
         <inertia ixx="0.0017389750000000002" ixy="0" ixz="0"
@@ -18,5 +16,5 @@
     </link>
     <joint name="${tf_prefix}attach_joint" type="fixed">
-      <origin xyz="0 0 ${adapter_offset}" rpy="0 0 0"/>
+      <origin xyz="0 0 0" rpy="0 0 0"/>
       <parent link="${tf_prefix}base_link"/>
       <child link="${tf_prefix}tool_link"/>
@@ -30,20 +28,20 @@
                  izz="0.000001"/>
       </inertial>
-      <visual>
-        <origin xyz="0 0 ${adapter_offset / 2}" rpy="0 0 0"/>
+      <visual name="axia_ft_sensor_visual">
+        <origin xyz="0 0 0.0" rpy="0 0 0"/>
         <geometry>
-          <cylinder length="${adapter_offset}" radius="0.041"/>
+          <mesh filename="package://aic_assets/models/Axia80 M20/axia_ft_sensor_visual.glb"/>
         </geometry>
       </visual>
-      <collision name="collision1">
-        <origin xyz="0 0 ${adapter_offset / 2}" rpy="0 0 0"/>
+      <collision name="axia80_m20_collider_cylinder">
+        <origin xyz="0.0 -0.000004 0.012699" rpy="3.141593 0.0 0.0"/>
         <geometry>
-          <cylinder length="${adapter_offset}" radius="0.041"/>
+          <cylinder length="0.025399" radius="0.041519"/>
         </geometry>
       </collision>
-      <collision name="collision2">
-        <origin xyz="-0.0475 0 0.0075" rpy="0 0 0"/>
+      <collision name="axia80_m20001_collider_cylinder">
+        <origin xyz="0.0 0.041828 0.018432" rpy="-1.570796 0 0"/>
         <geometry>
-          <box size="0.015 0.015 0.015"/>
+          <cylinder radius="0.006027" length="0.016717"/>
         </geometry>
       </collision>
@@ -103,21 +101,4 @@
       </sensor>
     </gazebo>
-    <gazebo reference="${tf_prefix}tool_link">
-      <sensor name="contact_sensor" type="contact">
-        <contact>
-          <!-- The reason for the convoluted collision name reference is due to URDF to SDF
-          conversion prepending and appending names to the collision name. The current workaround
-          is provide an exact name -->
-          <collision>${tf_prefix}tool_link_fixed_joint_lump__collision1_collision</collision>
-          <topic>collision/tool_link</topic>
-        </contact>
-      </sensor>
-      <!-- Reduce contact stiffness and damping for better stability -->
-      <kp>100000</kp>
-      <kd>100</kd>
-      <!-- Reduce friction in order to get smoother simulated force -->
-      <mu1>0.01</mu1>
-      <mu2>0.01</mu2>
-    </gazebo>
   </xacro:macro>
 </robot>

File: aic_description/urdf/ur_gz.urdf.xacro (robot description, xacro)
@@ -6,5 +6,8 @@
   <xacro:include filename="$(find ur_description)/urdf/ur_macro.xacro"/>
   <!-- import ATI Axia80-M20 macro -->
-  <xacro:include filename="$(find aic_assets)/models/ATI_Axia80_M20/axia80_m20_macro.xacro"/>
+  <xacro:include filename="$(find aic_assets)/models/Axia80 M20/axia80_m20_macro.xacro"/>
+  <xacro:include filename="$(find aic_assets)/models/Tri Cam Mount/tri_cam_mount_macro.xacro"/>
+  <xacro:include filename="$(find aic_assets)/models/Basler Camera/basler_camera_macro.xacro"/>
+  <xacro:include filename="$(find aic_assets)/models/Robotiq Hand-E/robotiq_hande_macro.xacro"/>
   <!-- <xacro:include filename="$(find ur_simulation_gz)/urdf/ur_gz.ros2_control.xacro" /> -->
   <xacro:include filename="$(find ur_description)/urdf/inc/ur_joint_control.xacro" />
@@ -25,4 +28,9 @@
   <xacro:arg name="ros_namespace" default="" />
   <xacro:arg name="ati_tf_prefix" default="ati/" />
+  <xacro:arg name="cam_mount_tf_prefix" default="cam_mount/" />
+  <xacro:arg name="wrist_camera_1_tf_prefix" default="wrist_camera_1/"/>
+  <xacro:arg name="wrist_camera_2_tf_prefix" default="wrist_camera_2/"/>
+  <xacro:arg name="wrist_camera_3_tf_prefix" default="wrist_camera_3/"/>
+  <xacro:arg name="gripper_tf_prefix" default="gripper/"/>
   <!-- Pose arguments for robot positioning -->
   <xacro:arg name="x" default="0.0" />
@@ -96,12 +104,48 @@
   <!-- ATI Force Torque sensor -->
   <xacro:axia80_m20
-    name="ati"
     tf_prefix="$(arg ati_tf_prefix)"
     >
   </xacro:axia80_m20>
+  <!-- Tri Cam Mount -->
+  <xacro:tri_cam_mount
+    tf_prefix="$(arg cam_mount_tf_prefix)"
+    >
+  </xacro:tri_cam_mount>
+  <xacro:basler_camera
+    tf_prefix="$(arg wrist_camera_1_tf_prefix)"
+    >
+  </xacro:basler_camera>
+  <xacro:basler_camera
+    tf_prefix="$(arg wrist_camera_2_tf_prefix)"
+    >
+  </xacro:basler_camera>
+  <xacro:robotiq_hand_e
+    tf_prefix="$(arg gripper_tf_prefix)"
+    >
+  </xacro:robotiq_hand_e>
+  <joint name="attach_tri_cam_mount" type="fixed">
+    <origin xyz="0 0 0" rpy="0 0 0"/>
+    <parent link="$(arg tf_prefix)tool0"/>
+    <child link="$(arg cam_mount_tf_prefix)cam_mount_link"/>
+  </joint>
   <joint name="attach_ft_sensor_joint" type="fixed">
-    <origin rpy="0 0 0" xyz="0 0 0"/>
-    <parent link="$(arg tf_prefix)tool0"/>
+    <origin xyz="0 0 0.0265" rpy="0 0 0"/>
+    <parent link="$(arg cam_mount_tf_prefix)cam_mount_link"/>
     <child link="$(arg ati_tf_prefix)base_link"/>
+  </joint>
+  <joint name="attach_wrist_camera_1" type="fixed">
+    <origin xyz="0.10395 0 0.054483" rpy="0.261799 0 -1.5708"/>
+    <parent link="$(arg cam_mount_tf_prefix)cam_mount_link"/>
+    <child link="$(arg wrist_camera_1_tf_prefix)basler_cam_link"/>
+  </joint>
+  <joint name="attach_wrist_camera_2" type="fixed">
+    <origin  xyz="-0.051975 -0.090023 0.054483" rpy="0.261799 0 2.61799"/>
+    <parent link="$(arg cam_mount_tf_prefix)cam_mount_link"/>
+    <child link="$(arg wrist_camera_2_tf_prefix)basler_cam_link"/>
+  </joint>
+  <joint name="attach_gripper" type="fixed">
+    <origin xyz="0 0 0.0519" rpy="0 0 0"/>
+    <parent link="$(arg cam_mount_tf_prefix)cam_mount_link"/>
+    <child link="$(arg gripper_tf_prefix)hande_base_link"/>
   </joint>
   <!-- ros2 control instance -->
@@ -122,5 +166,5 @@
       initial_positions="${dict(
         shoulder_pan_joint=0.0,
-        shoulder_lift_joint=-1.8645,
+        shoulder_lift_joint=-1.2645,
         elbow_joint=-2.35,
         wrist_1_joint=-0.5,

Commit message: add gripper action and fix joint and mesh transforms. Added gazebo camera plugins. Change from ogre2 to ogre so that distortion can be rendered.

File: aic_assets/models/Axia80 M20/axia80_m20_macro.xacro (robot description, xacro)
@@ -4,5 +4,5 @@
   <xacro:property name="tf_prefix" value="ati/"/>
   <!-- adapter_offset is the effective length that the adapter adds to the endeffector -->
-  <!-- <xacro:property name="adapter_offset" value="0.0245"/> -->
+  <xacro:property name="adapter_offset" value="0.0245"/>
   <xacro:macro name="axia80_m20" params="tf_prefix">
     <link name="${tf_prefix}base_link">
@@ -14,20 +14,6 @@
                  izz="0.0002521499999999999"/>
       </inertial>
-    </link>
-    <joint name="${tf_prefix}attach_joint" type="fixed">
-      <origin xyz="0 0 0" rpy="0 0 0"/>
-      <parent link="${tf_prefix}base_link"/>
-      <child link="${tf_prefix}tool_link"/>
-    </joint>
-    <link name="${tf_prefix}tool_link">
-      <inertial>
+      <visual name="axia_ft_sensor_visual">
         <origin xyz="0 0 0" rpy="0 0 0"/>
-        <mass value="0.001"/>
-        <inertia ixx="0.000001" ixy="0" ixz="0"
-                 iyy="0.000001" iyz="0"
-                 izz="0.000001"/>
-      </inertial>
-      <visual name="axia_ft_sensor_visual">
-        <origin xyz="0 0 0.0" rpy="0 0 0"/>
         <geometry>
           <mesh filename="package://aic_assets/models/Axia80 M20/axia_ft_sensor_visual.glb"/>
@@ -46,4 +32,18 @@
         </geometry>
       </collision>
+    </link>
+    <joint name="${tf_prefix}attach_joint" type="fixed">
+      <origin xyz="0 0 ${adapter_offset}" rpy="0 0 0"/>
+      <parent link="${tf_prefix}base_link"/>
+      <child link="${tf_prefix}tool_link"/>
+    </joint>
+    <link name="${tf_prefix}tool_link">
+      <inertial>
+        <origin xyz="0 0 0" rpy="0 0 0"/>
+        <mass value="0.001"/>
+        <inertia ixx="0.000001" ixy="0" ixz="0"
+                 iyy="0.000001" iyz="0"
+                 izz="0.000001"/>
+      </inertial>
     </link>
     <gazebo reference="${tf_prefix}attach_joint">

File: aic_assets/models/Basler Camera/basler_camera_macro.xacro (robot description, xacro)
@@ -1,9 +1,15 @@
 <?xml version="1.0"?>
 <robot xmlns:xacro="http://wiki.ros.org/xacro">
-  <!-- TF prefix parameter -->
-  <xacro:property name="tf_prefix" value="wrist_camera_1/"/>
-  <xacro:macro name="basler_camera" params="tf_prefix">
+  <xacro:macro name="basler_camera" params="name tf_prefix cam_lens_offset use_sim_cam">
     <link name="${tf_prefix}basler_cam_link">
+      <inertial>
+        <origin xyz="0 0 0" rpy="0 0 0"/>
+        <mass value="0.1"/>
+        <inertia ixx="0.00002083" ixy="0" ixz="0"
+                 iyy="0.00002083" iyz="0"
+                 izz="0.000015"/>
+      </inertial>
       <visual name="basler_cam_visual">
+        <origin xyz="0 0 -${cam_lens_offset}" rpy="0 0 0"/>
         <geometry>
           <mesh filename="package://aic_assets/models/Basler Camera/basler_cam_visual.glb"/>
@@ -11,5 +17,5 @@
       </visual>
       <collision name="lens001_collider_cylinder">
-        <origin xyz="-0.000005 0.000001 0.013336" rpy="0.0 0.0 0.0"/>
+        <origin xyz="-0.000005 0.000001 ${0.013336 - cam_lens_offset}" rpy="0.0 0.0 0.0"/>
         <geometry>
           <cylinder radius="0.016429" length="0.040108"/>
@@ -17,5 +23,5 @@
       </collision>
       <collision name="basler_ace2_gige027_collider_box">
-        <origin xyz="-0.000001 -0.000017 -0.031178" rpy="0.0 0.0 0.0"/>
+        <origin xyz="-0.000001 -0.000017 ${-0.031178 - cam_lens_offset}" rpy="0.0 0.0 0.0"/>
         <geometry>
           <box size="0.028998 0.028965 0.04919"/>
@@ -23,5 +29,5 @@
       </collision>
       <collision name="basler_ace2_gige011_collider_cylinder">
-        <origin xyz="-0.005773 -0.0081 -0.058082" rpy="0.0 0.0 0.0"/>
+        <origin xyz="-0.005773 -0.0081 ${-0.058082 - cam_lens_offset}" rpy="0.0 0.0 0.0"/>
         <geometry>
           <cylinder radius="0.005145" length="0.008255"/>
@@ -29,4 +35,67 @@
       </collision>
     </link>
+    <link name="${tf_prefix}sensor_link">
+      <!-- inertial property required for valid conversion to SDF,
+        so we set a tiny mass and M.O.I. here -->
+      <inertial>
+        <origin xyz="0 0 0" rpy="0 0 0"/>
+        <mass value="0.001"/>
+        <inertia ixx="0.000001" ixy="0" ixz="0"
+                 iyy="0.000001" iyz="0"
+                 izz="0.000001"/>
+      </inertial>
+    </link>
+    <joint name="${tf_prefix}attach_sensor" type="fixed">
+      <origin xyz="0 0 0" rpy="0 0 0"/>
+      <parent link="${tf_prefix}basler_cam_link"/>
+      <child link="${tf_prefix}sensor_link"/>
+    </joint>
+    <gazebo reference="${tf_prefix}attach_sensor">
+      <preserveFixedJoint>true</preserveFixedJoint>
+    </gazebo>
+    <xacro:if value="${use_sim_cam}">
+      <gazebo reference="${tf_prefix}sensor_link">
+        <sensor name="${name}" type="camera">
+          <pose>0 0 0 1.57079632679 -1.57079632679 0</pose>
+          <update_rate>10.0</update_rate>
+          <topic>/${name}/image</topic>
+          <always_on>true</always_on>
+          <visualize>true</visualize>
+          <frame_id>${tf_prefix}sensor_link</frame_id>
+          <camera name="${name}">
+            <camera_info_topic>/${name}/camera_info</camera_info_topic>
+            <image>
+              <width>1936</width>
+              <height>1216</height>
+              <format>R8G8B8</format>
+            </image>
+            <lens>
+              <intrinsics>
+                <fx>1426.0899369363822</fx>
+                <fy>1425.8803490609369</fy>
+                <cx>971.4830445595597</cx>
+                <cy>609.4634452956738</cy>
+              </intrinsics>
+            </lens>
+            <clip>
+              <near>0.02</near>
+              <far>300</far>
+            </clip>
+            <distortion>
+              <k1>-0.17436234247184138</k1>
+              <k2>0.12925824906602892</k2>
+              <k3>-0.04034799597244948</k3>
+              <p1>0.0002735332847870008</p1>
+              <p2>-0.00021180159916717322</p2>
+            </distortion>
+            <noise>
+              <type>gaussian</type>
+              <mean>0.0</mean>
+              <stddev>0.007</stddev>
+            </noise>
+          </camera>
+        </sensor>
+      </gazebo>
+    </xacro:if>
   </xacro:macro>
 </robot>

File: aic_assets/models/Robotiq Hand-E/robotiq_hande_macro.xacro (robot description, xacro)
@@ -11,4 +11,11 @@
     />
     <link name="${tf_prefix}hande_base_link">
+      <inertial>
+        <origin xyz="0 0 0" rpy="0 0 0"/>
+        <mass value="1.0"/>
+        <inertia ixx="0.1" ixy="0" ixz="0"
+                 iyy="0.1" iyz="0"
+                 izz="0.1"/>
+      </inertial>
       <visual name="hande_base_visual">
         <origin xyz="0 0 0" rpy="0 0 0"/>
@@ -31,4 +38,11 @@
     </link>
     <link name="${tf_prefix}hande_finger_link_l">
+      <inertial>
+        <origin xyz="0 0 0" rpy="0 0 0"/>
+        <mass value="0.2"/>
+        <inertia ixx="0.0001" ixy="0" ixz="0"
+                 iyy="0.00009" iyz="0"
+                 izz="0.00003"/>
+      </inertial>
       <visual name="hande_finger_visual">
         <origin xyz="0 0 0" rpy="0 0 0"/>
@@ -63,11 +77,18 @@
       <inertial>
         <origin xyz="0 0 0" rpy="0 0 0"/>
-        <mass value="0.03804"/>
-        <inertia ixx="1E-9" ixy="0.0" ixz="0.0" iyy="1E-9" iyz="0.0" izz="1E-9"/>
+        <mass value="0.2"/>
+        <inertia ixx="0.0001" ixy="0.0" ixz="0.0" iyy="0.00009" iyz="0.0" izz="0.00003"/>
       </inertial>
     </link>
     <link name="${tf_prefix}hande_finger_link_r">
+      <inertial>
+        <origin xyz="0 0 0" rpy="0 0 0"/>
+        <mass value="0.2"/>
+        <inertia ixx="0.0001" ixy="0" ixz="0"
+                 iyy="0.00009" iyz="0"
+                 izz="0.00003"/>
+      </inertial>
       <visual name="hande_finger_visual">
-        <origin xyz="0 0 0" rpy="0 0 ${pi}"/>
+        <origin xyz="0 0 0" rpy="0 0 3.14157"/>
         <geometry>
           <mesh filename="package://aic_assets/models/Robotiq Hand-E/hande_finger_visual.glb"/>
@@ -75,5 +96,5 @@
       </visual>
       <collision name="finger_collider_box">
-        <origin xyz="0.032595 -0.00001 0.138138" rpy="0.0 0.0 ${pi}"/>
+        <origin xyz="-0.032595 -0.00001 0.138138" rpy="0.0 0.0 0.0"/>
         <geometry>
           <box size="0.007839 0.021 0.028622"/>
@@ -81,5 +102,5 @@
       </collision>
       <collision name="finger_collider_box001">
-        <origin xyz="0.028 -0.00001 0.16145" rpy="0.0 0.0 ${pi}"/>
+        <origin xyz="-0.028 -0.00001 0.16145" rpy="0.0 0.0 0.0"/>
         <geometry>
           <box size="0.006 0.021 0.021498"/>
@@ -87,5 +108,5 @@
       </collision>
       <collision name="finger_collider_box002">
-        <origin xyz="0.014354 -0.015 0.124725" rpy="0.0 0.0 ${pi}"/>
+        <origin xyz="-0.014354 -0.015 0.124725" rpy="0.0 0.0 0.0"/>
         <geometry>
           <box size="0.044319 0.0075 0.003949"/>
@@ -93,5 +114,5 @@
       </collision>
       <collision name="finger_collider_box003">
-        <origin xyz="0.027046 -0.00954 0.129064" rpy="0.0 0.0 ${pi}"/>
+        <origin xyz="-0.027046 -0.00954 0.129064" rpy="0.0 0.0 0.0"/>
         <geometry>
           <box size="0.017387 0.018419 0.009271"/>
@@ -100,6 +121,6 @@
       <inertial>
         <origin xyz="0 0 0" rpy="0 0 0"/>
-        <mass value="0.03804"/>
-        <inertia ixx="1E-9" ixy="0.0" ixz="0.0" iyy="1E-9" iyz="0.0" izz="1E-9"/>
+        <mass value="0.2"/>
+        <inertia ixx="0.0001" ixy="0.0" ixz="0.0" iyy="0.00009" iyz="0.0" izz="0.00003"/>
       </inertial>
     </link>

File: aic_assets/models/Tri Cam Mount/tri_cam_mount_macro.xacro (robot description, xacro)
@@ -4,4 +4,11 @@
   <xacro:macro name="tri_cam_mount" params="tf_prefix">
     <link name="${tf_prefix}cam_mount_link">
+      <inertial>
+        <origin xyz="0 0 0" rpy="0 0 0"/>
+        <mass value="0.001"/>
+        <inertia ixx="0.000001" ixy="0" ixz="0"
+                 iyy="0.000001" iyz="0"
+                 izz="0.000001"/>
+      </inertial>
       <visual name="cam_mount_visual">
         <geometry>

File: aic_description/urdf/ur_gz.urdf.xacro (robot description, xacro)
@@ -12,4 +12,5 @@
   <!-- <xacro:include filename="$(find ur_simulation_gz)/urdf/ur_gz.ros2_control.xacro" /> -->
   <xacro:include filename="$(find ur_description)/urdf/inc/ur_joint_control.xacro" />
+  <xacro:property name="D2R" value="${pi / 180.0}"/>
   <!-- possible 'ur_type' values: ur3, ur5, ur10, ur3e, ur5e, ur7e, ur10e, ur12e, ur16e, ur8long, ur15, ur20, ur30 -->
   <!-- the default value should raise an error in case this was called without defining the type -->
@@ -33,4 +34,8 @@
   <xacro:arg name="wrist_camera_3_tf_prefix" default="wrist_camera_3/"/>
   <xacro:arg name="gripper_tf_prefix" default="gripper/"/>
+  <xacro:arg name="cam_lens_offset" default="0.035" />
+  <xacro:arg name="cam_mount_offset" default="0.09495" />
+  <!-- If true, enable Gazebo camera in sim -->
+  <xacro:arg name="use_sim_cam" default="${True}"/>
   <!-- Pose arguments for robot positioning -->
   <xacro:arg name="x" default="0.0" />
@@ -40,7 +45,4 @@
   <xacro:arg name="pitch" default="0.0" />
   <xacro:arg name="yaw" default="0.0" />
-  <xacro:property name="adapter_offset" value="0.0254"/>
-  <!-- <xacro:arg name="adapter_offset" default="0.0254" />
-  <xacro:arg name="adapter_offset_halved" default="0.0127" /> -->
   <!-- create link fixed to the "world" -->
   <link name="world" />
@@ -113,9 +115,22 @@
   </xacro:tri_cam_mount>
   <xacro:basler_camera
+    name="wrist_camera_1"
     tf_prefix="$(arg wrist_camera_1_tf_prefix)"
+    cam_lens_offset="$(arg cam_lens_offset)"
+    use_sim_cam="$(arg use_sim_cam)"
     >
   </xacro:basler_camera>
   <xacro:basler_camera
+    name="wrist_camera_2"
     tf_prefix="$(arg wrist_camera_2_tf_prefix)"
+    cam_lens_offset="$(arg cam_lens_offset)"
+    use_sim_cam="$(arg use_sim_cam)"
+    >
+  </xacro:basler_camera>
+  <xacro:basler_camera
+    name="wrist_camera_3"
+    tf_prefix="$(arg wrist_camera_3_tf_prefix)"
+    cam_lens_offset="$(arg cam_lens_offset)"
+    use_sim_cam="$(arg use_sim_cam)"
     >
   </xacro:basler_camera>
@@ -141,16 +156,24 @@
   </joint>
   <joint name="attach_wrist_camera_1" type="fixed">
-    <origin xyz="0.10395 0 0.054483" rpy="0.261799 0 -1.5708"/>
+    <origin xyz="$(arg cam_mount_offset) 0 ${0.054483+$(arg cam_lens_offset)}"
+      rpy="0.261799 0 -1.5708"/>
     <parent link="$(arg cam_mount_tf_prefix)cam_mount_link"/>
     <child link="$(arg wrist_camera_1_tf_prefix)basler_cam_link"/>
   </joint>
   <joint name="attach_wrist_camera_2" type="fixed">
-    <origin  xyz="-0.051975 -0.090023 0.054483" rpy="0.261799 0 2.61799"/>
+    <origin xyz="-${$(arg cam_mount_offset) * sin(30.0*D2R)} -${$(arg cam_mount_offset) * cos(30.0*D2R)} ${0.054483+$(arg cam_lens_offset)}"
+      rpy="0.261799 0 2.61799"/>
     <parent link="$(arg cam_mount_tf_prefix)cam_mount_link"/>
     <child link="$(arg wrist_camera_2_tf_prefix)basler_cam_link"/>
   </joint>
+  <joint name="attach_wrist_camera_3" type="fixed">
+    <origin xyz="-${$(arg cam_mount_offset) * sin(30.0*D2R)} ${$(arg cam_mount_offset) * cos(30.0*D2R)} ${0.054483+$(arg cam_lens_offset)}"
+      rpy="0.261799 0 0.523599"/>
+    <parent link="$(arg cam_mount_tf_prefix)cam_mount_link"/>
+    <child link="$(arg wrist_camera_3_tf_prefix)basler_cam_link"/>
+  </joint>
   <joint name="attach_gripper" type="fixed">
-    <origin xyz="0 0 0.0519" rpy="0 0 0"/>
-    <parent link="$(arg cam_mount_tf_prefix)cam_mount_link"/>
+    <origin xyz="0 0 0" rpy="0 0 0"/>
+    <parent link="$(arg ati_tf_prefix)tool_link"/>
     <child link="$(arg gripper_tf_prefix)hande_base_link"/>
   </joint>
