Commit message: add gripper controller and state/command interfaces to gripper

File: aic_assets/models/Robotiq Hand-E/robotiq_hande_macro.xacro (robot description, xacro)
@@ -1,9 +1,13 @@
 <?xml version="1.0"?>
 <robot xmlns:xacro="http://wiki.ros.org/xacro">
-  <xacro:property name="tf_prefix" value="gripper/"/>
-  <xacro:property name="grip_pos_min" value="0"/>
-  <xacro:property name="grip_pos_max" value="0.025"/>
-  <xacro:property name="hande_height" value="0.099"/>
-  <xacro:macro name="robotiq_hand_e" params="tf_prefix">
+  <xacro:include filename="$(find aic_assets)/models/Robotiq Hand-E/robotiq_hande.ros2_control.xacro"/>
+  <xacro:macro name="robotiq_hande" params="name tf_prefix grip_pos_min grip_pos_max grip_vel_max grip_effort_max initial_pos">
+    <xacro:robotiq_hande_ros2_control
+      name="${name}"
+      tf_prefix="${tf_prefix}"
+      grip_pos_min="${grip_pos_min}"
+      grip_pos_max="${grip_pos_max}"
+      initial_pos="${initial_pos}"
+    />
     <link name="${tf_prefix}hande_base_link">
       <visual name="hande_base_visual">
@@ -26,11 +30,4 @@
       </collision>
     </link>
-    <joint name="${tf_prefix}robotiq_hande_left_finger_joint" type="prismatic">
-      <origin xyz="0 0 0" rpy="0 0 0"/>
-      <parent link="${tf_prefix}hande_base_link"/>
-      <child link="${tf_prefix}hande_finger_link_l"/>
-      <axis xyz="1 0 0"/>
-      <limit effort="130" lower="${grip_pos_min}" upper="${grip_pos_max}" velocity="0.15"/>
-    </joint>
     <link name="${tf_prefix}hande_finger_link_l">
       <visual name="hande_finger_visual">
@@ -70,12 +67,4 @@
       </inertial>
     </link>
-    <joint name="${tf_prefix}robotiq_hande_right_finger_joint" type="prismatic">
-      <origin xyz="0 0 ${hande_height}" rpy="0 0 0"/>
-      <parent link="${tf_prefix}hande_base_link"/>
-      <child link="${tf_prefix}hande_finger_link_r"/>
-      <axis xyz="-1 0 0"/>
-      <limit effort="130" lower="${grip_pos_min}" upper="${grip_pos_max}" velocity="0.15"/>
-      <mimic joint="${tf_prefix}robotiq_hande_left_finger_joint" multiplier="1" offset="0"/>
-    </joint>
     <link name="${tf_prefix}hande_finger_link_r">
       <visual name="hande_finger_visual">
@@ -115,4 +104,25 @@
       </inertial>
     </link>
+    <joint name="${tf_prefix}left_finger_joint" type="prismatic">
+      <origin xyz="0 0 0" rpy="0 0 0"/>
+      <parent link="${tf_prefix}hande_base_link"/>
+      <child link="${tf_prefix}hande_finger_link_l"/>
+      <axis xyz="1 0 0"/>
+      <limit effort="${grip_effort_max}" lower="${grip_pos_min}" upper="${grip_pos_max}" velocity="${grip_vel_max}"/>
+    </joint>
+    <joint name="${tf_prefix}right_finger_joint" type="prismatic">
+      <origin xyz="0 0 0" rpy="0 0 0"/>
+      <parent link="${tf_prefix}hande_base_link"/>
+      <child link="${tf_prefix}hande_finger_link_r"/>
+      <axis xyz="-1 0 0"/>
+      <limit effort="${grip_effort_max}" lower="${grip_pos_min}" upper="${grip_pos_max}" velocity="${grip_vel_max}"/>
+      <mimic joint="${tf_prefix}left_finger_joint" multiplier="1" offset="0"/>
+    </joint>
+    <link name="${tf_prefix}tool_frame"/>
+    <joint name="${tf_prefix}attach_tool_frame" type="fixed">
+      <origin xyz="0 0 0.128" rpy="0 0 0"/>
+      <parent link="${tf_prefix}hande_base_link"/>
+      <child link="${tf_prefix}tool_frame"/>
+    </joint>
   </xacro:macro>
 </robot>

File: aic_description/urdf/ur_gz.urdf.xacro (robot description, xacro)
@@ -120,8 +120,14 @@
     >
   </xacro:basler_camera>
-  <xacro:robotiq_hand_e
+  <xacro:robotiq_hande
+    name="gripper"
     tf_prefix="$(arg gripper_tf_prefix)"
+    grip_pos_min="0.0"
+    grip_pos_max="0.025"
+    grip_vel_max="0.05"
+    grip_effort_max="130"
+    initial_pos="0.025"
     >
-  </xacro:robotiq_hand_e>
+  </xacro:robotiq_hande>
   <joint name="attach_tri_cam_mount" type="fixed">
     <origin xyz="0 0 0" rpy="0 0 0"/>

Commit message: Offset visual and collision finger geometries

File: aic_assets/models/Robotiq Hand-E/robotiq_hande_macro.xacro (robot description, xacro)
@@ -12,4 +12,5 @@
       initial_pos="${initial_pos}"
     />
+    <xacro:property name="gripper_jaw_offset" value="0.025"/>
     <link name="${tf_prefix}hande_base_link">
       <inertial>
@@ -48,5 +49,5 @@
       </inertial>
       <visual name="hande_finger_visual">
-        <origin xyz="0 0 0" rpy="0 0 0"/>
+        <origin xyz="${-gripper_jaw_offset} 0 0" rpy="0 0 0"/>
         <geometry>
           <mesh filename="package://aic_assets/models/Robotiq Hand-E/hande_finger_visual.glb"/>
@@ -54,5 +55,5 @@
       </visual>
       <collision name="finger_collider_box">
-        <origin xyz="0.032595 -0.00001 0.138138" rpy="0.0 0.0 0.0"/>
+        <origin xyz="${-gripper_jaw_offset + 0.032595} -0.00001 0.138138" rpy="0.0 0.0 0.0"/>
         <geometry>
           <box size="0.007839 0.021 0.028622"/>
@@ -60,5 +61,5 @@
       </collision>
       <collision name="finger_collider_box001">
-        <origin xyz="0.028 -0.00001 0.16145" rpy="0.0 0.0 0.0"/>
+        <origin xyz="${-gripper_jaw_offset + 0.028} -0.00001 0.16145" rpy="0.0 0.0 0.0"/>
         <geometry>
           <box size="0.006 0.021 0.021498"/>
@@ -66,5 +67,5 @@
       </collision>
       <collision name="finger_collider_box002">
-        <origin xyz="0.014354 -0.015 0.124725" rpy="0.0 0.0 0.0"/>
+        <origin xyz="${-gripper_jaw_offset + 0.014354} -0.015 0.124725" rpy="0.0 0.0 0.0"/>
         <geometry>
           <box size="0.044319 0.0075 0.003949"/>
@@ -72,5 +73,5 @@
       </collision>
       <collision name="finger_collider_box003">
-        <origin xyz="0.027046 -0.00954 0.129064" rpy="0.0 0.0 0.0"/>
+        <origin xyz="${-gripper_jaw_offset + 0.027046} -0.00954 0.129064" rpy="0.0 0.0 0.0"/>
         <geometry>
           <box size="0.017387 0.018419 0.009271"/>
@@ -92,5 +93,5 @@
       </inertial>
       <visual name="hande_finger_visual">
-        <origin xyz="0 0 0" rpy="0 0 3.14157"/>
+        <origin xyz="${gripper_jaw_offset} 0 0" rpy="0 0 3.14157"/>
         <geometry>
           <mesh filename="package://aic_assets/models/Robotiq Hand-E/hande_finger_visual.glb"/>
@@ -98,5 +99,5 @@
       </visual>
       <collision name="finger_collider_box">
-        <origin xyz="-0.032595 -0.00001 0.138138" rpy="0.0 0.0 0.0"/>
+        <origin xyz="${gripper_jaw_offset - 0.032595} -0.00001 0.138138" rpy="0.0 0.0 0.0"/>
         <geometry>
           <box size="0.007839 0.021 0.028622"/>
@@ -104,5 +105,5 @@
       </collision>
       <collision name="finger_collider_box001">
-        <origin xyz="-0.028 -0.00001 0.16145" rpy="0.0 0.0 0.0"/>
+        <origin xyz="${gripper_jaw_offset - 0.028} -0.00001 0.16145" rpy="0.0 0.0 0.0"/>
         <geometry>
           <box size="0.006 0.021 0.021498"/>
@@ -110,5 +111,5 @@
       </collision>
       <collision name="finger_collider_box002">
-        <origin xyz="-0.014354 -0.015 0.124725" rpy="0.0 0.0 0.0"/>
+        <origin xyz="${gripper_jaw_offset - 0.014354} -0.015 0.124725" rpy="0.0 0.0 0.0"/>
         <geometry>
           <box size="0.044319 0.0075 0.003949"/>
@@ -116,5 +117,5 @@
       </collision>
       <collision name="finger_collider_box003">
-        <origin xyz="-0.027046 -0.00954 0.129064" rpy="0.0 0.0 0.0"/>
+        <origin xyz="${gripper_jaw_offset - 0.027046} -0.00954 0.129064" rpy="0.0 0.0 0.0"/>
         <geometry>
           <box size="0.017387 0.018419 0.009271"/>
@@ -144,5 +145,5 @@
     <link name="${tf_prefix}tool_frame"/>
     <joint name="${tf_prefix}attach_tool_frame" type="fixed">
-      <origin xyz="0 0 0.128" rpy="0 0 0"/>
+      <origin xyz="0 0 0.172" rpy="0 0 0"/>
       <parent link="${tf_prefix}hande_base_link"/>
       <child link="${tf_prefix}tool_frame"/>

File: aic_description/urdf/ur_gz.urdf.xacro (robot description, xacro)
@@ -135,5 +135,5 @@
     grip_effort_min="20"
     grip_effort_max="130"
-    initial_pos="0.025"
+    initial_pos="0.02"
     >
   </xacro:robotiq_hande>
