Commit message: Fix transforms in aic_robot and gripper

File: aic_assets/models/Robotiq Hand-E/robotiq_hande.ros2_control.xacro (robot description, xacro)
@@ -1,8 +1,8 @@
 <?xml version="1.0"?>
 <robot xmlns:xacro="http://wiki.ros.org/xacro">
-  <xacro:macro name="robotiq_hande_ros2_control" params="name tf_prefix grip_pos_min grip_pos_max grip_effort_min grip_effort_max initial_pos">
+  <xacro:macro name="robotiq_hande_ros2_control" params="name tf_prefix grip_pos_min grip_pos_max grip_effort_min grip_effort_max initial_pos hardware_plugin:='gz_ros2_control/GazeboSimSystem'">
     <ros2_control name="${name}" type="system">
       <hardware>
-        <plugin>gz_ros2_control/GazeboSimSystem</plugin>
+        <plugin>${hardware_plugin}</plugin>
       </hardware>
       <joint name="${tf_prefix}left_finger_joint">

File: aic_assets/models/Robotiq Hand-E/robotiq_hande_macro.xacro (robot description, xacro)
@@ -2,5 +2,5 @@
 <robot xmlns:xacro="http://wiki.ros.org/xacro">
   <xacro:include filename="$(find aic_assets)/models/Robotiq Hand-E/robotiq_hande.ros2_control.xacro"/>
-  <xacro:macro name="robotiq_hande" params="name tf_prefix grip_pos_min grip_pos_max grip_vel_max grip_effort_min grip_effort_max initial_pos">
+  <xacro:macro name="robotiq_hande" params="name tf_prefix grip_pos_min grip_pos_max grip_vel_max grip_effort_min grip_effort_max initial_pos hardware_plugin:='gz_ros2_control/GazeboSimSystem'">
     <xacro:robotiq_hande_ros2_control
       name="${name}"
@@ -11,4 +11,5 @@
       grip_effort_max="${grip_effort_max}"
       initial_pos="${initial_pos}"
+      hardware_plugin="${hardware_plugin}"
     />
     <xacro:property name="gripper_jaw_offset" value="0.025"/>

File: aic_description/urdf/ur_gz.urdf.xacro (robot description, xacro)
@@ -36,4 +36,5 @@
   <xacro:arg name="gripper_tf_prefix" default="gripper/"/>
   <xacro:arg name="gripper_initial_pos" default="0.00655"/>
+  <xacro:arg name="gripper_hardware_plugin" default="gz_ros2_control/GazeboSimSystem"/>
   <xacro:arg name="cam_mount_radial_offset" default="0.1" />
   <xacro:arg name="cam_mount_axial_offset" default="0.08" />
@@ -153,4 +154,5 @@
     grip_effort_max="130"
     initial_pos="$(arg gripper_initial_pos)"
+    hardware_plugin="$(arg gripper_hardware_plugin)"
     >
   </xacro:robotiq_hande>

Commit message: Cleanup gripper hardware interface switch between simulators

File: aic_assets/models/Robotiq Hand-E/robotiq_hande.ros2_control.xacro (robot description, xacro)
@@ -1,5 +1,5 @@
 <?xml version="1.0"?>
 <robot xmlns:xacro="http://wiki.ros.org/xacro">
-  <xacro:macro name="robotiq_hande_ros2_control" params="name tf_prefix grip_pos_min grip_pos_max grip_effort_min grip_effort_max initial_pos hardware_plugin:='gz_ros2_control/GazeboSimSystem'">
+  <xacro:macro name="robotiq_hande_ros2_control" params="name tf_prefix grip_pos_min grip_pos_max grip_effort_min grip_effort_max initial_pos hardware_plugin">
     <ros2_control name="${name}" type="system">
       <hardware>

File: aic_assets/models/Robotiq Hand-E/robotiq_hande_macro.xacro (robot description, xacro)
@@ -1,5 +1,16 @@
 <?xml version="1.0"?>
 <robot xmlns:xacro="http://wiki.ros.org/xacro">
-  <xacro:macro name="robotiq_hande" params="name tf_prefix grip_pos_min grip_pos_max grip_vel_max grip_effort_min grip_effort_max initial_pos">
+  <xacro:include filename="$(find aic_assets)/models/Robotiq Hand-E/robotiq_hande.ros2_control.xacro"/>
+  <xacro:macro name="robotiq_hande" params="name tf_prefix grip_pos_min grip_pos_max grip_vel_max grip_effort_min grip_effort_max initial_pos hardware_plugin">
+    <xacro:robotiq_hande_ros2_control
+      name="${name}"
+      tf_prefix="${tf_prefix}"
+      grip_pos_min="${grip_pos_min}"
+      grip_pos_max="${grip_pos_max}"
+      grip_effort_min="${grip_effort_min}"
+      grip_effort_max="${grip_effort_max}"
+      initial_pos="${initial_pos}"
+      hardware_plugin="${hardware_plugin}"
+    />
     <xacro:property name="gripper_jaw_offset" value="0.025"/>
     <link name="${tf_prefix}hande_base_link">

File: aic_description/config/gazebo_ros2_control.xacro (robot description, xacro)
@@ -24,34 +24,4 @@
         wrist_3_joint=1.4110)}"
     />
-    <!-- Gripper joints -->
-    <joint name="$(arg gripper_tf_prefix)left_finger_joint">
-      <command_interface name="position">
-        <param name="min">0.0</param>
-        <param name="max">0.025</param>
-      </command_interface>
-      <command_interface name="effort">
-        <param name="min">20</param>
-        <param name="max">130</param>
-      </command_interface>
-      <state_interface name="position">
-        <param name="initial_value">$(arg gripper_initial_pos)</param>
-      </state_interface>
-      <state_interface name="velocity">
-        <param name="initial_value">0.0</param>
-      </state_interface>
-      <state_interface name="effort">
-        <param name="initial_value">0.0</param>
-      </state_interface>
-    </joint>
-    <joint name="$(arg gripper_tf_prefix)right_finger_joint">
-      <param name="mimic">$(arg gripper_tf_prefix)left_finger_joint</param>
-      <param name="multiplier">1</param>
-      <state_interface name="position">
-        <param name="initial_value">$(arg gripper_initial_pos)</param>
-      </state_interface>
-      <state_interface name="velocity">
-        <param name="initial_value">0.0</param>
-      </state_interface>
-    </joint>
   </ros2_control>
 </robot>

File: aic_description/urdf/ur_gz.urdf.xacro (robot description, xacro)
@@ -36,4 +36,5 @@
   <xacro:arg name="gripper_tf_prefix" default="gripper/"/>
   <xacro:arg name="gripper_initial_pos" default="0.00655"/>
+  <xacro:arg name="hardware_plugin" default="gz_ros2_control/GazeboSimSystem"/>
   <xacro:arg name="cam_mount_radial_offset" default="0.1" />
   <xacro:arg name="cam_mount_axial_offset" default="0.08" />
@@ -153,4 +154,5 @@
     grip_effort_max="130"
     initial_pos="$(arg gripper_initial_pos)"
+    hardware_plugin="$(arg hardware_plugin)"
     >
   </xacro:robotiq_hande>

File: aic_utils/aic_mujoco/config/mujoco_ros2_control.xacro (robot description, xacro)
@@ -26,24 +26,4 @@
         wrist_3_joint=1.4110)}"
     />
-    <!-- Gripper joints -->
-    <joint name="$(arg gripper_tf_prefix)left_finger_joint">
-      <command_interface name="position">
-        <param name="min">0.0</param>
-        <param name="max">0.025</param>
-      </command_interface>
-      <command_interface name="effort">
-        <param name="min">0.5</param>
-        <param name="max">5</param>
-      </command_interface>
-      <state_interface name="position">
-        <param name="initial_value">$(arg gripper_initial_pos)</param>
-      </state_interface>
-      <state_interface name="velocity">
-        <param name="initial_value">0.0</param>
-      </state_interface>
-      <state_interface name="effort">
-        <param name="initial_value">0.0</param>
-      </state_interface>
-    </joint>
   </ros2_control>
 </robot>

Commit message: Remove mimic joint from controller

File: aic_assets/models/Robotiq Hand-E/robotiq_hande.ros2_control.xacro (robot description, xacro)
@@ -25,14 +25,4 @@
         </state_interface>
       </joint>
-      <joint name="${tf_prefix}right_finger_joint">
-        <param name="mimic">${tf_prefix}left_finger_joint</param>
-        <param name="multiplier">1</param>
-        <state_interface name="position">
-          <param name="initial_value">${initial_pos}</param>
-        </state_interface>
-        <state_interface name="velocity">
-          <param name="initial_value">0.0</param>
-        </state_interface>
-      </joint>
     </ros2_control>
   </xacro:macro>

Commit message: Remove mimic joint from controller, address review comments

File: aic_assets/models/Robotiq Hand-E/robotiq_hande.ros2_control.xacro (robot description, xacro)
@@ -1,5 +1,5 @@
 <?xml version="1.0"?>
 <robot xmlns:xacro="http://wiki.ros.org/xacro">
-  <xacro:macro name="robotiq_hande_ros2_control" params="name tf_prefix grip_pos_min grip_pos_max grip_effort_min grip_effort_max initial_pos hardware_plugin">
+  <xacro:macro name="robotiq_hande_ros2_control" params="name tf_prefix grip_pos_min grip_pos_max grip_effort_min grip_effort_max initial_pos hardware_plugin:='gz_ros2_control/GazeboSimSystem'">
     <ros2_control name="${name}" type="system">
       <hardware>

File: aic_description/urdf/ur_gz.urdf.xacro (robot description, xacro)
@@ -37,5 +37,5 @@
   <xacro:arg name="gripper_initial_pos" default="0.00655"/>
   <xacro:arg name="hardware_plugin" default="gz_ros2_control/GazeboSimSystem"/>
-  <xacro:arg name="cam_mount_radial_offset" default="0.1" />
+    <xacro:arg name="cam_mount_radial_offset" default="0.1" />
   <xacro:arg name="cam_mount_axial_offset" default="0.08" />
   <!-- If true, enable Gazebo camera in sim -->

Commit message: Minimize diff with main

File: aic_assets/models/Robotiq Hand-E/robotiq_hande.ros2_control.xacro (robot description, xacro)
@@ -1,8 +1,11 @@
 <?xml version="1.0"?>
 <robot xmlns:xacro="http://wiki.ros.org/xacro">
-  <xacro:macro name="robotiq_hande_ros2_control" params="name tf_prefix grip_pos_min grip_pos_max grip_effort_min grip_effort_max initial_pos hardware_plugin:='gz_ros2_control/GazeboSimSystem'">
+  <!-- Declare hardware_plugin as a global xacro arg with Gazebo default.
+       MuJoCo launch overrides this via: hardware_plugin:=mujoco_ros2_control/MujocoSystem -->
+  <xacro:arg name="hardware_plugin" default="gz_ros2_control/GazeboSimSystem"/>
+  <xacro:macro name="robotiq_hande_ros2_control" params="name tf_prefix grip_pos_min grip_pos_max grip_effort_min grip_effort_max initial_pos">
     <ros2_control name="${name}" type="system">
       <hardware>
-        <plugin>${hardware_plugin}</plugin>
+        <plugin>$(arg hardware_plugin)</plugin>
       </hardware>
       <joint name="${tf_prefix}left_finger_joint">

File: aic_assets/models/Robotiq Hand-E/robotiq_hande_macro.xacro (robot description, xacro)
@@ -2,5 +2,5 @@
 <robot xmlns:xacro="http://wiki.ros.org/xacro">
   <xacro:include filename="$(find aic_assets)/models/Robotiq Hand-E/robotiq_hande.ros2_control.xacro"/>
-  <xacro:macro name="robotiq_hande" params="name tf_prefix grip_pos_min grip_pos_max grip_vel_max grip_effort_min grip_effort_max initial_pos hardware_plugin">
+  <xacro:macro name="robotiq_hande" params="name tf_prefix grip_pos_min grip_pos_max grip_vel_max grip_effort_min grip_effort_max initial_pos">
     <xacro:robotiq_hande_ros2_control
       name="${name}"
@@ -11,5 +11,4 @@
       grip_effort_max="${grip_effort_max}"
       initial_pos="${initial_pos}"
-      hardware_plugin="${hardware_plugin}"
     />
     <xacro:property name="gripper_jaw_offset" value="0.025"/>

File: aic_description/urdf/ur_gz.urdf.xacro (robot description, xacro)
@@ -36,6 +36,5 @@
   <xacro:arg name="gripper_tf_prefix" default="gripper/"/>
   <xacro:arg name="gripper_initial_pos" default="0.00655"/>
-  <xacro:arg name="hardware_plugin" default="gz_ros2_control/GazeboSimSystem"/>
-    <xacro:arg name="cam_mount_radial_offset" default="0.1" />
+  <xacro:arg name="cam_mount_radial_offset" default="0.1" />
   <xacro:arg name="cam_mount_axial_offset" default="0.08" />
   <!-- If true, enable Gazebo camera in sim -->
@@ -154,5 +153,4 @@
     grip_effort_max="130"
     initial_pos="$(arg gripper_initial_pos)"
-    hardware_plugin="$(arg hardware_plugin)"
     >
   </xacro:robotiq_hande>
