Commit message: add force torque sensor and move_to_contact script
add move_to_contact script

Move move_to_contact to separate launch file

Signed-off-by: Yadunund <yadunund@intrinsic.ai>

Tweak script and robot initial pos

Signed-off-by: Yadunund <yadunund@intrinsic.ai>

Create ATI asset

Signed-off-by: Yadunund <yadunund@intrinsic.ai>

File: aic_description/urdf/ur_gz.urdf.xacro (robot description, xacro)
@@ -3,6 +3,8 @@
   <!-- robot name parameter -->
   <xacro:arg name="name" default="ur"/>
-  <!-- import main macro -->
+  <!-- import UR macro -->
   <xacro:include filename="$(find ur_description)/urdf/ur_macro.xacro"/>
+  <!-- import ATI Axia80-M20 macro -->
+  <xacro:include filename="$(find aic_assets)/models/ATI_Axia80_M20/axia80_m20_macro.xacro"/>
   <!-- <xacro:include filename="$(find ur_simulation_gz)/urdf/ur_gz.ros2_control.xacro" /> -->
   <xacro:include filename="$(find ur_description)/urdf/inc/ur_joint_control.xacro" />
@@ -22,4 +24,5 @@
   <xacro:arg name="simulation_controllers" default="" />
   <xacro:arg name="ros_namespace" default="" />
+  <xacro:arg name="ati_tf_prefix" default="ati/" />
   <!-- Pose arguments for robot positioning -->
   <xacro:arg name="x" default="0.0" />
@@ -29,8 +32,17 @@
   <xacro:arg name="pitch" default="0.0" />
   <xacro:arg name="yaw" default="0.0" />
+  <xacro:property name="adapter_offset" value="0.0254"/>
+  <!-- <xacro:arg name="adapter_offset" default="0.0254" />
+  <xacro:arg name="adapter_offset_halved" default="0.0127" /> -->
   <!-- create link fixed to the "world" -->
   <link name="world" />
-  <link name="ground_plane">
-    <!-- <visual>
+  <link name="tabletop" />
+  <joint name="tabletop_joint" type="fixed">
+    <origin xyz="$(arg x) $(arg y) $(arg z)" rpy="$(arg roll) $(arg pitch) $(arg yaw)" />
+    <parent link="world"/>
+    <child link="tabletop"/>
+  </joint>
+  <!-- <link name="ground_plane">
+    <visual>
       <origin rpy="0 0 0" xyz="0 0 0"/>
       <geometry>
@@ -40,5 +52,5 @@
         <color rgba="1 1 1 0.5"/>
       </material>
-    </visual> -->
+    </visual>
     <collision>
       <origin rpy="0 0 0" xyz="0 0 0"/>
@@ -52,10 +64,10 @@
     <parent link="world"/>
     <child link="ground_plane"/>
-  </joint>
+  </joint> -->
   <!-- arm -->
   <xacro:ur_robot
     name="$(arg name)"
     tf_prefix="$(arg tf_prefix)"
-    parent="ground_plane"
+    parent="tabletop"
     joint_limits_parameters_file="$(arg joint_limit_params)"
     kinematics_parameters_file="$(arg kinematics_params)"
@@ -82,16 +94,15 @@
     </plugin>
   </gazebo>
-  <gazebo reference="$(arg tf_prefix)wrist_3_joint">
-    <sensor name="force_torque_sensor" type="force_torque">
-      <always_on>true</always_on>
-      <update_rate>50</update_rate>
-      <visualize>true</visualize>
-      <topic>$(arg tf_prefix)wrist_3_joint/force_torque</topic>
-      <force_torque>
-        <frame>sensor</frame>
-        <measure_direction>parent_to_child</measure_direction>
-      </force_torque>
-    </sensor>
-  </gazebo>
+  <!-- ATI Force Torque sensor -->
+  <xacro:axia80_m20
+    name="ati"
+    tf_prefix="$(arg ati_tf_prefix)"
+    >
+  </xacro:axia80_m20>
+  <joint name="attach_ft_sensor_joint" type="fixed">
+    <origin rpy="0 0 0" xyz="0 0 0"/>
+    <parent link="$(arg tf_prefix)tool0"/>
+    <child link="$(arg ati_tf_prefix)base_link"/>
+  </joint>
   <!-- ros2 control instance -->
   <ros2_control name="GazeboSystem" type="system">
@@ -99,5 +110,5 @@
       <plugin>gz_ros2_control/GazeboSimSystem</plugin>
     </hardware>
-    <sensor name="force_torque_sensor" type="force_torque">
+    <sensor name="AtiForceTorqueSensor" type="force_torque">
       <state_interface name="force.x"/>
       <state_interface name="force.y"/>
@@ -109,5 +120,5 @@
     <xacro:ur_joint_control_description
       tf_prefix="$(arg tf_prefix)"
-      initial_positions="${dict(shoulder_pan_joint=0.0,shoulder_lift_joint=-1.57,elbow_joint=0.0,wrist_1_joint=-1.57,wrist_2_joint=0.0,wrist_3_joint=0.0)}"
+      initial_positions="${dict(shoulder_pan_joint=0.0,shoulder_lift_joint=-1.571,elbow_joint=-1.571,wrist_1_joint=-1.571,wrist_2_joint=1.5708,wrist_3_joint=0.0)}"
     />
   </ros2_control>

Commit message: Remove third wrist camera

File: aic_description/urdf/ur_gz.urdf.xacro (robot description, xacro)
@@ -32,5 +32,4 @@
   <xacro:arg name="wrist_camera_1_tf_prefix" default="wrist_camera_1/"/>
   <xacro:arg name="wrist_camera_2_tf_prefix" default="wrist_camera_2/"/>
-  <xacro:arg name="wrist_camera_3_tf_prefix" default="wrist_camera_3/"/>
   <xacro:arg name="gripper_tf_prefix" default="gripper/"/>
   <xacro:arg name="cam_lens_offset" default="0.035" />
@@ -128,11 +127,4 @@
     >
   </xacro:basler_camera>
-  <xacro:basler_camera
-    name="wrist_camera_3"
-    tf_prefix="$(arg wrist_camera_3_tf_prefix)"
-    cam_lens_offset="$(arg cam_lens_offset)"
-    use_sim_cam="$(arg use_sim_cam)"
-    >
-  </xacro:basler_camera>
   <xacro:robotiq_hande
     name="gripper"
@@ -167,10 +159,4 @@
     <child link="$(arg wrist_camera_2_tf_prefix)basler_cam_link"/>
   </joint>
-  <joint name="attach_wrist_camera_3" type="fixed">
-    <origin xyz="-${$(arg cam_mount_offset) * sin(30.0*D2R)} ${$(arg cam_mount_offset) * cos(30.0*D2R)} ${0.054483+$(arg cam_lens_offset)}"
-      rpy="0.261799 0 0.523599"/>
-    <parent link="$(arg cam_mount_tf_prefix)cam_mount_link"/>
-    <child link="$(arg wrist_camera_3_tf_prefix)basler_cam_link"/>
-  </joint>
   <joint name="attach_gripper" type="fixed">
     <origin xyz="0 0 0" rpy="0 0 0"/>

Commit message: move second wrist camera to 120 degree rotation from first camera

File: aic_description/urdf/ur_gz.urdf.xacro (robot description, xacro)
@@ -35,5 +35,4 @@
   <xacro:arg name="cam_mount_radial_offset" default="0.1" />
   <xacro:arg name="cam_mount_axial_offset" default="0.08" />
-  <xacro:arg name="cam_mount_stereo_baseline" default="0.04" />
   <!-- If true, enable Gazebo camera in sim -->
   <xacro:arg name="use_sim_cam" default="${True}"/>
@@ -147,6 +146,6 @@
     <child link="$(arg ati_tf_prefix)base_link"/>
   </joint>
-  <!-- Dummy link to simplify all the composite rotations -->
-  <link name="wrist_camera_intermediate_link">
+  <!-- Dummy link to simplify the chain of rotations -->
+  <link name="wrist_camera_1_intermediate_link">
     <inertial>
       <origin xyz="0 0 0" rpy="0 0 0"/>
@@ -161,14 +160,30 @@
       rpy="${90.0*D2R} ${-90.0*D2R} ${0.0*D2R}"/>
     <parent link="$(arg cam_mount_tf_prefix)cam_mount_link"/>
-    <child link="wrist_camera_intermediate_link"/>
+    <child link="wrist_camera_1_intermediate_link"/>
   </joint>
   <joint name="attach_wrist_camera_1" type="fixed">
     <origin xyz="0 0 0" rpy="${0.0*D2R} ${15.0*D2R} ${0.0*D2R}"/>
-    <parent link="wrist_camera_intermediate_link"/>
+    <parent link="wrist_camera_1_intermediate_link"/>
     <child link="$(arg wrist_camera_1_tf_prefix)basler_cam_link"/>
   </joint>
+  <!-- Dummy link to simplify the chain of rotations -->
+  <link name="wrist_camera_2_intermediate_link">
+    <inertial>
+      <origin xyz="0 0 0" rpy="0 0 0"/>
+      <mass value="0.001"/>
+      <inertia ixx="0.000001" ixy="0" ixz="0"
+               iyy="0.000001" iyz="0"
+               izz="0.000001"/>
+    </inertial>
+  </link>
+  <joint name="wrist_camera_2_intermediate_joint" type="fixed">
+    <origin xyz="${-cos(30.0*D2R)*$(arg cam_mount_radial_offset)} ${sin(30.0*D2R)*$(arg cam_mount_radial_offset)} $(arg cam_mount_axial_offset)"
+      rpy="${90.0*D2R} ${-90.0*D2R} ${-120.0*D2R}"/>
+    <parent link="$(arg cam_mount_tf_prefix)cam_mount_link"/>
+    <child link="wrist_camera_2_intermediate_link"/>
+  </joint>
   <joint name="attach_wrist_camera_2" type="fixed">
-    <origin xyz="0 -$(arg cam_mount_stereo_baseline) 0" rpy="${0.0*D2R} ${15.0*D2R} ${0.0*D2R}"/>
-    <parent link="wrist_camera_intermediate_link"/>
+    <origin xyz="0 0 0" rpy="${0.0*D2R} ${15.0*D2R} ${0.0*D2R}"/>
+    <parent link="wrist_camera_2_intermediate_link"/>
     <child link="$(arg wrist_camera_2_tf_prefix)basler_cam_link"/>
   </joint>

Commit message: rename the cameras: left, center, right

File: aic_description/urdf/ur_gz.urdf.xacro (robot description, xacro)
@@ -30,7 +30,7 @@
   <xacro:arg name="ati_tf_prefix" default="ati/" />
   <xacro:arg name="cam_mount_tf_prefix" default="cam_mount/" />
-  <xacro:arg name="wrist_camera_1_tf_prefix" default="wrist_camera_1/"/>
-  <xacro:arg name="wrist_camera_2_tf_prefix" default="wrist_camera_2/"/>
-  <xacro:arg name="wrist_camera_3_tf_prefix" default="wrist_camera_3/"/>
+  <xacro:arg name="left_camera_tf_prefix" default="left_camera/"/>
+  <xacro:arg name="center_camera_tf_prefix" default="center_camera/"/>
+  <xacro:arg name="right_camera_tf_prefix" default="right_camera/"/>
   <xacro:arg name="gripper_tf_prefix" default="gripper/"/>
   <xacro:arg name="gripper_initial_pos" default="0.012"/>
@@ -124,18 +124,18 @@
   </xacro:camera_mount>
   <xacro:basler_camera
-    name="wrist_camera_1"
-    tf_prefix="$(arg wrist_camera_1_tf_prefix)"
+    name="left_camera"
+    tf_prefix="$(arg left_camera_tf_prefix)"
     use_sim_cam="$(arg use_sim_cam)"
     >
   </xacro:basler_camera>
   <xacro:basler_camera
-    name="wrist_camera_2"
-    tf_prefix="$(arg wrist_camera_2_tf_prefix)"
+    name="center_camera"
+    tf_prefix="$(arg center_camera_tf_prefix)"
     use_sim_cam="$(arg use_sim_cam)"
     >
   </xacro:basler_camera>
   <xacro:basler_camera
-    name="wrist_camera_3"
-    tf_prefix="$(arg wrist_camera_3_tf_prefix)"
+    name="right_camera"
+    tf_prefix="$(arg right_camera_tf_prefix)"
     use_sim_cam="$(arg use_sim_cam)"
     >
@@ -152,7 +152,4 @@
     >
   </xacro:robotiq_hande>
- <!-- ********************
-      ** wrist_camera_1 **
-      ******************** -->
   <joint name="attach_cam_mount" type="fixed">
     <origin xyz="0 0 -.0265" rpy="0 0 0"/>
@@ -165,24 +162,27 @@
     <child link="$(arg ati_tf_prefix)base_link"/>
   </joint>
-  <joint name="attach_wrist_camera_1" type="fixed">
+  <!-- *******************
+       ** center_camera **
+       ******************* -->
+  <joint name="attach_center_camera" type="fixed">
     <origin xyz="0 -0.1077 -.00719" rpy="0 -1.30899630 1.57079623"/>
     <parent link="$(arg cam_mount_tf_prefix)cam_mount_link"/>
-    <child link="$(arg wrist_camera_1_tf_prefix)camera_link"/>
-  </joint>
-  <!-- ********************
-       ** wrist_camera_2 **
-       ******************** -->
-  <joint name="attach_wrist_camera_2" type="fixed">
+    <child link="$(arg center_camera_tf_prefix)camera_link"/>
+  </joint>
+  <!-- *****************
+       ** left_camera **
+       ***************** -->
+  <joint name="attach_left_camera" type="fixed">
     <origin xyz="-0.09326 -0.053843 -0.007188" rpy="0 -1.30899630 0.523599027"/>
     <parent link="$(arg cam_mount_tf_prefix)cam_mount_link"/>
-    <child link="$(arg wrist_camera_2_tf_prefix)camera_link"/>
-  </joint>
-  <!-- ********************
-       ** wrist_camera_3 **
-       ******************** -->
-  <joint name="attach_wrist_camera_3" type="fixed">
+    <child link="$(arg left_camera_tf_prefix)camera_link"/>
+  </joint>
+  <!-- ******************
+       ** right_camera **
+       ****************** -->
+  <joint name="attach_right_camera" type="fixed">
     <origin xyz="0.09326 -0.053843 -0.007188" rpy="0 -1.30899630 2.61799343"/>
     <parent link="$(arg cam_mount_tf_prefix)cam_mount_link"/>
-    <child link="$(arg wrist_camera_3_tf_prefix)camera_link"/>
+    <child link="$(arg right_camera_tf_prefix)camera_link"/>
   </joint>
   <joint name="attach_gripper" type="fixed">
