Commit message: Include xacros for each component
Signed-off-by: Yadunund <yadunund@intrinsic.ai>

File: aic_description/urdf/task_board.urdf.xacro (robot description, xacro)
@@ -1,4 +1,11 @@
 <?xml version="1.0"?>
 <robot xmlns:xacro="http://wiki.ros.org/xacro" name="task_board">
+  <!-- Include component macros -->
+  <xacro:include filename="$(find aic_assets)/models/Task Board Base/task_board_base_macro.xacro"/>
+  <xacro:include filename="$(find aic_assets)/models/LC Mount/lc_mount_macro.xacro"/>
+  <xacro:include filename="$(find aic_assets)/models/SFP Mount/sfp_mount_macro.xacro"/>
+  <xacro:include filename="$(find aic_assets)/models/SC Mount/sc_mount_macro.xacro"/>
+  <xacro:include filename="$(find aic_assets)/models/SC Port/sc_port_macro.xacro"/>
+  <xacro:include filename="$(find aic_assets)/models/NIC Card Mount/nic_card_mount_macro.xacro"/>
   <!-- Task Board Base pose arguments -->
   <xacro:arg name="x" default="-0.2"/>
@@ -63,21 +70,7 @@
   <!-- Task Board Base is at (0.25, 0, 1.14) relative to world in original SDF -->
   <!-- Components are positioned relative to base -->
-  <!-- Base link for the entire task board assembly -->
-  <link name="task_board_base_link">
-    <inertial>
-      <mass value="5.0"/>
-      <inertia ixx="0.1" ixy="0.0" ixz="0.0" iyy="0.1" iyz="0.0" izz="0.1"/>
-    </inertial>
-  </link>
-  <gazebo reference="task_board_base_link">
-    <visual>
-      <geometry>
-        <mesh>
-          <uri>model://Task Board Base</uri>
-        </mesh>
-      </geometry>
-    </visual>
-  </gazebo>
-  <!-- LC Mount 01 -->
+  <!-- Instantiate Task Board Base -->
+  <xacro:task_board_base prefix="task_board_"/>  <!-- LC Mount 01 -->
+  <xacro:lc_mount prefix="lc_mount_01_"/>
   <joint name="lc_mount_01_joint" type="fixed">
     <parent link="task_board_base_link"/>
@@ -85,20 +78,6 @@
     <origin xyz="${0.0215 + $(arg lc_mount_01_delta_x)} ${-0.10625 + $(arg lc_mount_01_delta_y)} ${0.01 + $(arg lc_mount_01_delta_z)}" rpy="0 0 0"/>
   </joint>
-  <link name="lc_mount_01_link">
-    <inertial>
-      <mass value="0.1"/>
-      <inertia ixx="0.001" ixy="0.0" ixz="0.0" iyy="0.001" iyz="0.0" izz="0.001"/>
-    </inertial>
-  </link>
-  <gazebo reference="lc_mount_01_link">
-    <visual>
-      <geometry>
-        <mesh>
-          <uri>model://LC Mount</uri>
-        </mesh>
-      </geometry>
-    </visual>
-  </gazebo>
   <!-- SFP Mount 01 -->
+  <xacro:sfp_mount prefix="sfp_mount_01_"/>
   <joint name="sfp_mount_01_joint" type="fixed">
     <parent link="task_board_base_link"/>
@@ -106,20 +85,6 @@
     <origin xyz="${0.0535 + $(arg sfp_mount_01_delta_x)} ${-0.10625 + $(arg sfp_mount_01_delta_y)} ${0.01 + $(arg sfp_mount_01_delta_z)}" rpy="0 0 0"/>
   </joint>
-  <link name="sfp_mount_01_link">
-    <inertial>
-      <mass value="0.1"/>
-      <inertia ixx="0.001" ixy="0.0" ixz="0.0" iyy="0.001" iyz="0.0" izz="0.001"/>
-    </inertial>
-  </link>
-  <gazebo reference="sfp_mount_01_link">
-    <visual>
-      <geometry>
-        <mesh>
-          <uri>model://SFP Mount</uri>
-        </mesh>
-      </geometry>
-    </visual>
-  </gazebo>
   <!-- SC Mount 01 -->
+  <xacro:sc_mount prefix="sc_mount_01_"/>
   <joint name="sc_mount_01_joint" type="fixed">
     <parent link="task_board_base_link"/>
@@ -127,20 +92,6 @@
     <origin xyz="${0.0985 + $(arg sc_mount_01_delta_x)} ${-0.10625 + $(arg sc_mount_01_delta_y)} ${0.01 + $(arg sc_mount_01_delta_z)}" rpy="0 0 0"/>
   </joint>
-  <link name="sc_mount_01_link">
-    <inertial>
-      <mass value="0.1"/>
-      <inertia ixx="0.001" ixy="0.0" ixz="0.0" iyy="0.001" iyz="0.0" izz="0.001"/>
-    </inertial>
-  </link>
-  <gazebo reference="sc_mount_01_link">
-    <visual>
-      <geometry>
-        <mesh>
-          <uri>model://SC Mount</uri>
-        </mesh>
-      </geometry>
-    </visual>
-  </gazebo>
   <!-- LC Mount 02 -->
+  <xacro:lc_mount prefix="lc_mount_02_"/>
   <joint name="lc_mount_02_joint" type="fixed">
     <parent link="task_board_base_link"/>
@@ -148,20 +99,6 @@
     <origin xyz="${0.0215 + $(arg lc_mount_02_delta_x)} ${0.10625 + $(arg lc_mount_02_delta_y)} ${0.01 + $(arg lc_mount_02_delta_z)}" rpy="0 0 0"/>
   </joint>
-  <link name="lc_mount_02_link">
-    <inertial>
-      <mass value="0.1"/>
-      <inertia ixx="0.001" ixy="0.0" ixz="0.0" iyy="0.001" iyz="0.0" izz="0.001"/>
-    </inertial>
-  </link>
-  <gazebo reference="lc_mount_02_link">
-    <visual>
-      <geometry>
-        <mesh>
-          <uri>model://LC Mount</uri>
-        </mesh>
-      </geometry>
-    </visual>
-  </gazebo>
   <!-- SFP Mount 02 -->
+  <xacro:sfp_mount prefix="sfp_mount_02_"/>
   <joint name="sfp_mount_02_joint" type="fixed">
     <parent link="task_board_base_link"/>
@@ -169,20 +106,6 @@
     <origin xyz="${0.0535 + $(arg sfp_mount_02_delta_x)} ${0.10625 + $(arg sfp_mount_02_delta_y)} ${0.01 + $(arg sfp_mount_02_delta_z)}" rpy="0 0 0"/>
   </joint>
-  <link name="sfp_mount_02_link">
-    <inertial>
-      <mass value="0.1"/>
-      <inertia ixx="0.001" ixy="0.0" ixz="0.0" iyy="0.001" iyz="0.0" izz="0.001"/>
-    </inertial>
-  </link>
-  <gazebo reference="sfp_mount_02_link">
-    <visual>
-      <geometry>
-        <mesh>
-          <uri>model://SFP Mount</uri>
-        </mesh>
-      </geometry>
-    </visual>
-  </gazebo>
   <!-- SC Mount 02 -->
+  <xacro:sc_mount prefix="sc_mount_02_"/>
   <joint name="sc_mount_02_joint" type="fixed">
     <parent link="task_board_base_link"/>
@@ -190,20 +113,6 @@
     <origin xyz="${0.0985 + $(arg sc_mount_02_delta_x)} ${0.10625 + $(arg sc_mount_02_delta_y)} ${0.01 + $(arg sc_mount_02_delta_z)}" rpy="0 0 0"/>
   </joint>
-  <link name="sc_mount_02_link">
-    <inertial>
-      <mass value="0.1"/>
-      <inertia ixx="0.001" ixy="0.0" ixz="0.0" iyy="0.001" iyz="0.0" izz="0.001"/>
-    </inertial>
-  </link>
-  <gazebo reference="sc_mount_02_link">
-    <visual>
-      <geometry>
-        <mesh>
-          <uri>model://SC Mount</uri>
-        </mesh>
-      </geometry>
-    </visual>
-  </gazebo>
   <!-- SC Port 01 -->
+  <xacro:sc_port prefix="sc_port_01_"/>
   <joint name="sc_port_01_joint" type="fixed">
     <parent link="task_board_base_link"/>
@@ -211,20 +120,6 @@
     <origin xyz="${-0.075 + $(arg sc_port_01_delta_x)} ${0.0295 + $(arg sc_port_01_delta_y)} ${0.01 + $(arg sc_port_01_delta_z)}" rpy="1.57 0 1.57"/>
   </joint>
-  <link name="sc_port_01_link">
-    <inertial>
-      <mass value="0.1"/>
-      <inertia ixx="0.001" ixy="0.0" ixz="0.0" iyy="0.001" iyz="0.0" izz="0.001"/>
-    </inertial>
-  </link>
-  <gazebo reference="sc_port_01_link">
-    <visual>
-      <geometry>
-        <mesh>
-          <uri>model://SC Port</uri>
-        </mesh>
-      </geometry>
-    </visual>
-  </gazebo>
   <!-- SC Port 02 -->
+  <xacro:sc_port prefix="sc_port_02_"/>
   <joint name="sc_port_02_joint" type="fixed">
     <parent link="task_board_base_link"/>
@@ -232,20 +127,6 @@
     <origin xyz="${-0.075 + $(arg sc_port_02_delta_x)} ${0.0705 + $(arg sc_port_02_delta_y)} ${0.01 + $(arg sc_port_02_delta_z)}" rpy="1.57 0 1.57"/>
   </joint>
-  <link name="sc_port_02_link">
-    <inertial>
-      <mass value="0.1"/>
-      <inertia ixx="0.001" ixy="0.0" ixz="0.0" iyy="0.001" iyz="0.0" izz="0.001"/>
-    </inertial>
-  </link>
-  <gazebo reference="sc_port_02_link">
-    <visual>
-      <geometry>
-        <mesh>
-          <uri>model://SC Port</uri>
-        </mesh>
-      </geometry>
-    </visual>
-  </gazebo>
   <!-- NIC Card Mount 01 -->
+  <xacro:nic_card_mount prefix="nic_card_mount_01_"/>
   <joint name="nic_card_mount_01_joint" type="fixed">
     <parent link="task_board_base_link"/>
@@ -253,20 +134,6 @@
     <origin xyz="${-0.081418 + $(arg nic_card_mount_01_delta_x)} ${-0.0145 + $(arg nic_card_mount_01_delta_y)} ${0.01 + $(arg nic_card_mount_01_delta_z)}" rpy="0 0 0"/>
   </joint>
-  <link name="nic_card_mount_01_link">
-    <inertial>
-      <mass value="0.1"/>
-      <inertia ixx="0.001" ixy="0.0" ixz="0.0" iyy="0.001" iyz="0.0" izz="0.001"/>
-    </inertial>
-  </link>
-  <gazebo reference="nic_card_mount_01_link">
-    <visual>
-      <geometry>
-        <mesh>
-          <uri>model://NIC Card Mount</uri>
-        </mesh>
-      </geometry>
-    </visual>
-  </gazebo>
   <!-- NIC Card Mount 02 -->
+  <xacro:nic_card_mount prefix="nic_card_mount_02_"/>
   <joint name="nic_card_mount_02_joint" type="fixed">
     <parent link="task_board_base_link"/>
@@ -274,20 +141,6 @@
     <origin xyz="${-0.081418 + $(arg nic_card_mount_02_delta_x)} ${-0.0545 + $(arg nic_card_mount_02_delta_y)} ${0.01 + $(arg nic_card_mount_02_delta_z)}" rpy="0 0 0"/>
   </joint>
-  <link name="nic_card_mount_02_link">
-    <inertial>
-      <mass value="0.1"/>
-      <inertia ixx="0.001" ixy="0.0" ixz="0.0" iyy="0.001" iyz="0.0" izz="0.001"/>
-    </inertial>
-  </link>
-  <gazebo reference="nic_card_mount_02_link">
-    <visual>
-      <geometry>
-        <mesh>
-          <uri>model://NIC Card Mount</uri>
-        </mesh>
-      </geometry>
-    </visual>
-  </gazebo>
   <!-- NIC Card Mount 03 -->
+  <xacro:nic_card_mount prefix="nic_card_mount_03_"/>
   <joint name="nic_card_mount_03_joint" type="fixed">
     <parent link="task_board_base_link"/>
@@ -295,20 +148,6 @@
     <origin xyz="${-0.081418 + $(arg nic_card_mount_03_delta_x)} ${-0.0945 + $(arg nic_card_mount_03_delta_y)} ${0.01 + $(arg nic_card_mount_03_delta_z)}" rpy="0 0 0"/>
   </joint>
-  <link name="nic_card_mount_03_link">
-    <inertial>
-      <mass value="0.1"/>
-      <inertia ixx="0.001" ixy="0.0" ixz="0.0" iyy="0.001" iyz="0.0" izz="0.001"/>
-    </inertial>
-  </link>
-  <gazebo reference="nic_card_mount_03_link">
-    <visual>
-      <geometry>
-        <mesh>
-          <uri>model://NIC Card Mount</uri>
-        </mesh>
-      </geometry>
-    </visual>
-  </gazebo>
   <!-- NIC Card Mount 04 -->
+  <xacro:nic_card_mount prefix="nic_card_mount_04_"/>
   <joint name="nic_card_mount_04_joint" type="fixed">
     <parent link="task_board_base_link"/>
@@ -316,20 +155,6 @@
     <origin xyz="${-0.081418 + $(arg nic_card_mount_04_delta_x)} ${-0.1345 + $(arg nic_card_mount_04_delta_y)} ${0.01 + $(arg nic_card_mount_04_delta_z)}" rpy="0 0 0"/>
   </joint>
-  <link name="nic_card_mount_04_link">
-    <inertial>
-      <mass value="0.1"/>
-      <inertia ixx="0.001" ixy="0.0" ixz="0.0" iyy="0.001" iyz="0.0" izz="0.001"/>
-    </inertial>
-  </link>
-  <gazebo reference="nic_card_mount_04_link">
-    <visual>
-      <geometry>
-        <mesh>
-          <uri>model://NIC Card Mount</uri>
-        </mesh>
-      </geometry>
-    </visual>
-  </gazebo>
   <!-- NIC Card Mount 05 -->
+  <xacro:nic_card_mount prefix="nic_card_mount_05_"/>
   <joint name="nic_card_mount_05_joint" type="fixed">
     <parent link="task_board_base_link"/>
@@ -337,18 +162,3 @@
     <origin xyz="${-0.081418 + $(arg nic_card_mount_05_delta_x)} ${-0.1745 + $(arg nic_card_mount_05_delta_y)} ${0.01 + $(arg nic_card_mount_05_delta_z)}" rpy="0 0 0"/>
   </joint>
-  <link name="nic_card_mount_05_link">
-    <inertial>
-      <mass value="0.1"/>
-      <inertia ixx="0.001" ixy="0.0" ixz="0.0" iyy="0.001" iyz="0.0" izz="0.001"/>
-    </inertial>
-  </link>
-  <gazebo reference="nic_card_mount_05_link">
-    <visual>
-      <geometry>
-        <mesh>
-          <uri>model://NIC Card Mount</uri>
-        </mesh>
-      </geometry>
-    </visual>
-  </gazebo>
 </robot>

Commit message: Fix convention for NIC rails and make spawning flexible
Signed-off-by: Yadunund <yadunund@intrinsic.ai>

File: aic_description/urdf/task_board.urdf.xacro (robot description, xacro)
@@ -47,24 +47,34 @@
   <xacro:arg name="sc_port_02_delta_y" default="0.0"/>
   <xacro:arg name="sc_port_02_delta_z" default="0.0"/>
+  <!-- NIC Card Mount 00 -->
+  <xacro:arg name="nic_card_mount_00_present" default="true"/>
+  <xacro:arg name="nic_card_mount_00_translation" default="0.0"/>
+  <xacro:arg name="nic_card_mount_00_roll" default="0.0"/>
+  <xacro:arg name="nic_card_mount_00_pitch" default="0.0"/>
+  <xacro:arg name="nic_card_mount_00_yaw" default="0.0"/>
   <!-- NIC Card Mount 01 -->
-  <xacro:arg name="nic_card_mount_01_delta_x" default="0.0"/>
-  <xacro:arg name="nic_card_mount_01_delta_y" default="0.0"/>
-  <xacro:arg name="nic_card_mount_01_delta_z" default="0.0"/>
+  <xacro:arg name="nic_card_mount_01_present" default="true"/>
+  <xacro:arg name="nic_card_mount_01_translation" default="0.0"/>
+  <xacro:arg name="nic_card_mount_01_roll" default="0.0"/>
+  <xacro:arg name="nic_card_mount_01_pitch" default="0.0"/>
+  <xacro:arg name="nic_card_mount_01_yaw" default="0.0"/>
   <!-- NIC Card Mount 02 -->
-  <xacro:arg name="nic_card_mount_02_delta_x" default="0.0"/>
-  <xacro:arg name="nic_card_mount_02_delta_y" default="0.0"/>
-  <xacro:arg name="nic_card_mount_02_delta_z" default="0.0"/>
+  <xacro:arg name="nic_card_mount_02_present" default="true"/>
+  <xacro:arg name="nic_card_mount_02_translation" default="0.0"/>
+  <xacro:arg name="nic_card_mount_02_roll" default="0.0"/>
+  <xacro:arg name="nic_card_mount_02_pitch" default="0.0"/>
+  <xacro:arg name="nic_card_mount_02_yaw" default="0.0"/>
   <!-- NIC Card Mount 03 -->
-  <xacro:arg name="nic_card_mount_03_delta_x" default="0.0"/>
-  <xacro:arg name="nic_card_mount_03_delta_y" default="0.0"/>
-  <xacro:arg name="nic_card_mount_03_delta_z" default="0.0"/>
+  <xacro:arg name="nic_card_mount_03_present" default="true"/>
+  <xacro:arg name="nic_card_mount_03_translation" default="0.0"/>
+  <xacro:arg name="nic_card_mount_03_roll" default="0.0"/>
+  <xacro:arg name="nic_card_mount_03_pitch" default="0.0"/>
+  <xacro:arg name="nic_card_mount_03_yaw" default="0.0"/>
   <!-- NIC Card Mount 04 -->
-  <xacro:arg name="nic_card_mount_04_delta_x" default="0.0"/>
-  <xacro:arg name="nic_card_mount_04_delta_y" default="0.0"/>
-  <xacro:arg name="nic_card_mount_04_delta_z" default="0.0"/>
-  <!-- NIC Card Mount 05 -->
-  <xacro:arg name="nic_card_mount_05_delta_x" default="0.0"/>
-  <xacro:arg name="nic_card_mount_05_delta_y" default="0.0"/>
-  <xacro:arg name="nic_card_mount_05_delta_z" default="0.0"/>
+  <xacro:arg name="nic_card_mount_04_present" default="true"/>
+  <xacro:arg name="nic_card_mount_04_translation" default="0.0"/>
+  <xacro:arg name="nic_card_mount_04_roll" default="0.0"/>
+  <xacro:arg name="nic_card_mount_04_pitch" default="0.0"/>
+  <xacro:arg name="nic_card_mount_04_yaw" default="0.0"/>
   <!-- Calculate absolute positions relative to task board base -->
   <!-- Task Board Base is at (0.25, 0, 1.14) relative to world in original SDF -->
@@ -127,39 +137,49 @@
     <origin xyz="${-0.075 + $(arg sc_port_02_delta_x)} ${0.0705 + $(arg sc_port_02_delta_y)} ${0.01 + $(arg sc_port_02_delta_z)}" rpy="1.57 0 1.57"/>
   </joint>
+  <!-- NIC Card Mount 00 (left-most) -->
+  <xacro:if value="$(arg nic_card_mount_00_present)">
+    <xacro:nic_card_mount prefix="nic_card_mount_00_"/>
+    <joint name="nic_card_mount_00_joint" type="fixed">
+      <parent link="task_board_base_link"/>
+      <child link="nic_card_mount_00_link"/>
+      <origin xyz="${-0.081418 + $(arg nic_card_mount_00_translation)} -0.1745 0.01" rpy="$(arg nic_card_mount_00_roll) $(arg nic_card_mount_00_pitch) $(arg nic_card_mount_00_yaw)"/>
+    </joint>
+  </xacro:if>
   <!-- NIC Card Mount 01 -->
-  <xacro:nic_card_mount prefix="nic_card_mount_01_"/>
-  <joint name="nic_card_mount_01_joint" type="fixed">
-    <parent link="task_board_base_link"/>
-    <child link="nic_card_mount_01_link"/>
-    <origin xyz="${-0.081418 + $(arg nic_card_mount_01_delta_x)} ${-0.0145 + $(arg nic_card_mount_01_delta_y)} ${0.01 + $(arg nic_card_mount_01_delta_z)}" rpy="0 0 0"/>
-  </joint>
-  <!-- NIC Card Mount 02 -->
-  <xacro:nic_card_mount prefix="nic_card_mount_02_"/>
-  <joint name="nic_card_mount_02_joint" type="fixed">
-    <parent link="task_board_base_link"/>
-    <child link="nic_card_mount_02_link"/>
-    <origin xyz="${-0.081418 + $(arg nic_card_mount_02_delta_x)} ${-0.0545 + $(arg nic_card_mount_02_delta_y)} ${0.01 + $(arg nic_card_mount_02_delta_z)}" rpy="0 0 0"/>
-  </joint>
+  <xacro:if value="$(arg nic_card_mount_01_present)">
+    <xacro:nic_card_mount prefix="nic_card_mount_01_"/>
+    <joint name="nic_card_mount_01_joint" type="fixed">
+      <parent link="task_board_base_link"/>
+      <child link="nic_card_mount_01_link"/>
+      <origin xyz="${-0.081418 + $(arg nic_card_mount_01_translation)} -0.1345 0.01" rpy="$(arg nic_card_mount_01_roll) $(arg nic_card_mount_01_pitch) $(arg nic_card_mount_01_yaw)"/>
+    </joint>
+  </xacro:if>
+  <!-- NIC Card Mount 02 (center) -->
+  <xacro:if value="$(arg nic_card_mount_02_present)">
+    <xacro:nic_card_mount prefix="nic_card_mount_02_"/>
+    <joint name="nic_card_mount_02_joint" type="fixed">
+      <parent link="task_board_base_link"/>
+      <child link="nic_card_mount_02_link"/>
+      <origin xyz="${-0.081418 + $(arg nic_card_mount_02_translation)} -0.0945 0.01" rpy="$(arg nic_card_mount_02_roll) $(arg nic_card_mount_02_pitch) $(arg nic_card_mount_02_yaw)"/>
+    </joint>
+  </xacro:if>
   <!-- NIC Card Mount 03 -->
-  <xacro:nic_card_mount prefix="nic_card_mount_03_"/>
-  <joint name="nic_card_mount_03_joint" type="fixed">
-    <parent link="task_board_base_link"/>
-    <child link="nic_card_mount_03_link"/>
-    <origin xyz="${-0.081418 + $(arg nic_card_mount_03_delta_x)} ${-0.0945 + $(arg nic_card_mount_03_delta_y)} ${0.01 + $(arg nic_card_mount_03_delta_z)}" rpy="0 0 0"/>
-  </joint>
-  <!-- NIC Card Mount 04 -->
-  <xacro:nic_card_mount prefix="nic_card_mount_04_"/>
-  <joint name="nic_card_mount_04_joint" type="fixed">
-    <parent link="task_board_base_link"/>
-    <child link="nic_card_mount_04_link"/>
-    <origin xyz="${-0.081418 + $(arg nic_card_mount_04_delta_x)} ${-0.1345 + $(arg nic_card_mount_04_delta_y)} ${0.01 + $(arg nic_card_mount_04_delta_z)}" rpy="0 0 0"/>
-  </joint>
-  <!-- NIC Card Mount 05 -->
-  <xacro:nic_card_mount prefix="nic_card_mount_05_"/>
-  <joint name="nic_card_mount_05_joint" type="fixed">
-    <parent link="task_board_base_link"/>
-    <child link="nic_card_mount_05_link"/>
-    <origin xyz="${-0.081418 + $(arg nic_card_mount_05_delta_x)} ${-0.1745 + $(arg nic_card_mount_05_delta_y)} ${0.01 + $(arg nic_card_mount_05_delta_z)}" rpy="0 0 0"/>
-  </joint>
+  <xacro:if value="$(arg nic_card_mount_03_present)">
+    <xacro:nic_card_mount prefix="nic_card_mount_03_"/>
+    <joint name="nic_card_mount_03_joint" type="fixed">
+      <parent link="task_board_base_link"/>
+      <child link="nic_card_mount_03_link"/>
+      <origin xyz="${-0.081418 + $(arg nic_card_mount_03_translation)} -0.0545 0.01" rpy="$(arg nic_card_mount_03_roll) $(arg nic_card_mount_03_pitch) $(arg nic_card_mount_03_yaw)"/>
+    </joint>
+  </xacro:if>
+  <!-- NIC Card Mount 04 (right-most) -->
+  <xacro:if value="$(arg nic_card_mount_04_present)">
+    <xacro:nic_card_mount prefix="nic_card_mount_04_"/>
+    <joint name="nic_card_mount_04_joint" type="fixed">
+      <parent link="task_board_base_link"/>
+      <child link="nic_card_mount_04_link"/>
+      <origin xyz="${-0.081418 + $(arg nic_card_mount_04_translation)} -0.0145 0.01" rpy="$(arg nic_card_mount_04_roll) $(arg nic_card_mount_04_pitch) $(arg nic_card_mount_04_yaw)"/>
+    </joint>
+  </xacro:if>
   <gazebo>
     <static>true</static>
