Commit message: updated necessary xacro files

File: aic_description/urdf/task_board.urdf.xacro (robot description, xacro)
@@ -106,5 +106,5 @@
       <parent link="task_board_base_link"/>
       <child link="lc_mount_rail_0_link"/>
-      <origin xyz="0.0275 ${-0.10625 + $(arg lc_mount_rail_0_translation)} 0.01" rpy="$(arg lc_mount_rail_0_roll) $(arg lc_mount_rail_0_pitch) $(arg lc_mount_rail_0_yaw)"/>
+      <origin xyz="0.01 ${-0.10625 + $(arg lc_mount_rail_0_translation)} 0.012" rpy="$(arg lc_mount_rail_0_roll) $(arg lc_mount_rail_0_pitch) $(arg lc_mount_rail_0_yaw)"/>
     </joint>
   </xacro:if>
@@ -115,5 +115,5 @@
       <parent link="task_board_base_link"/>
       <child link="sfp_mount_rail_0_link"/>
-      <origin xyz="0.0535 ${-0.10625 + $(arg sfp_mount_rail_0_translation)} 0.01" rpy="$(arg sfp_mount_rail_0_roll) $(arg sfp_mount_rail_0_pitch) $(arg sfp_mount_rail_0_yaw)"/>
+      <origin xyz="0.055 ${-0.10625 + $(arg sfp_mount_rail_0_translation)} 0.01" rpy="$(arg sfp_mount_rail_0_roll) $(arg sfp_mount_rail_0_pitch) $(arg sfp_mount_rail_0_yaw)"/>
     </joint>
   </xacro:if>
@@ -124,5 +124,5 @@
       <parent link="task_board_base_link"/>
       <child link="sc_mount_rail_0_link"/>
-      <origin xyz="0.0985 ${-0.10625 + $(arg sc_mount_rail_0_translation)} 0.01" rpy="$(arg sc_mount_rail_0_roll) $(arg sc_mount_rail_0_pitch) $(arg sc_mount_rail_0_yaw)"/>
+      <origin xyz="0.1 ${-0.10625 + $(arg sc_mount_rail_0_translation)} 0.012" rpy="$(arg sc_mount_rail_0_roll) $(arg sc_mount_rail_0_pitch) $(arg sc_mount_rail_0_yaw)"/>
     </joint>
   </xacro:if>
@@ -133,5 +133,5 @@
       <parent link="task_board_base_link"/>
       <child link="lc_mount_rail_1_link"/>
-      <origin xyz="0.0275 ${0.10625 + $(arg lc_mount_rail_1_translation)} 0.01" rpy="$(arg lc_mount_rail_1_roll) $(arg lc_mount_rail_1_pitch) $(arg lc_mount_rail_1_yaw)"/>
+      <origin xyz="0.01 ${0.10625 + $(arg lc_mount_rail_1_translation)} 0.012" rpy="$(arg lc_mount_rail_1_roll) $(arg lc_mount_rail_1_pitch) $(arg lc_mount_rail_1_yaw)"/>
     </joint>
   </xacro:if>
@@ -142,5 +142,5 @@
       <parent link="task_board_base_link"/>
       <child link="sfp_mount_rail_1_link"/>
-      <origin xyz="0.0535 ${0.10625 + $(arg sfp_mount_rail_1_translation)} 0.01" rpy="$(arg sfp_mount_rail_1_roll) $(arg sfp_mount_rail_1_pitch) $(arg sfp_mount_rail_1_yaw)"/>
+      <origin xyz="0.055 ${0.10625 + $(arg sfp_mount_rail_1_translation)} 0.01" rpy="$(arg sfp_mount_rail_1_roll) $(arg sfp_mount_rail_1_pitch) $(arg sfp_mount_rail_1_yaw)"/>
     </joint>
   </xacro:if>
@@ -156,5 +156,5 @@
   <!-- SC Port 0 -->
   <xacro:if value="$(arg sc_port_0_present)">
-    <xacro:sc_port prefix="sc_port_0" pose="${-0.075 + $(arg sc_port_0_translation)} 0.0295 0.0145 ${1.57 + $(arg sc_port_0_roll)} $(arg sc_port_0_pitch) ${1.57 + $(arg sc_port_0_yaw)}"/>
+    <xacro:sc_port prefix="sc_port_0" pose="${-0.075 + $(arg sc_port_0_translation)} 0.0295 0.0165 ${1.57 + $(arg sc_port_0_roll)} $(arg sc_port_0_pitch) ${1.57 + $(arg sc_port_0_yaw)}"/>
     <gazebo>
       <joint name="sc_port_0_joint" type="fixed">
@@ -166,5 +166,5 @@
   <!-- SC Port 1 -->
   <xacro:if value="$(arg sc_port_1_present)">
-    <xacro:sc_port prefix="sc_port_1" pose="${-0.075 + $(arg sc_port_1_translation)} 0.0705 0.0145 ${1.57 + $(arg sc_port_1_roll)} $(arg sc_port_1_pitch) ${1.57 + $(arg sc_port_1_yaw)}"/>
+    <xacro:sc_port prefix="sc_port_1" pose="${-0.075 + $(arg sc_port_1_translation)} 0.0705 0.0165 ${1.57 + $(arg sc_port_1_roll)} $(arg sc_port_1_pitch) ${1.57 + $(arg sc_port_1_yaw)}"/>
     <gazebo>
       <joint name="sc_port_1_joint" type="fixed">
@@ -176,5 +176,5 @@
   <!-- NIC Card Mount 0 (left-most) -->
   <xacro:if value="$(arg nic_card_mount_0_present)">
-    <xacro:nic_card_mount prefix="nic_card_mount_0" pose="${-0.081418 + $(arg nic_card_mount_0_translation)} -0.1745 0.01 $(arg nic_card_mount_0_roll) $(arg nic_card_mount_0_pitch) $(arg nic_card_mount_0_yaw)"/>
+    <xacro:nic_card_mount prefix="nic_card_mount_0" pose="${-0.081418 + $(arg nic_card_mount_0_translation)} -0.1745 0.012 $(arg nic_card_mount_0_roll) $(arg nic_card_mount_0_pitch) $(arg nic_card_mount_0_yaw)"/>
     <gazebo>
       <joint name="nic_card_mount_0_joint" type="fixed">
@@ -186,5 +186,5 @@
   <!-- NIC Card Mount 1 -->
   <xacro:if value="$(arg nic_card_mount_1_present)">
-    <xacro:nic_card_mount prefix="nic_card_mount_1" pose="${-0.081418 + $(arg nic_card_mount_1_translation)} -0.1345 0.01 $(arg nic_card_mount_1_roll) $(arg nic_card_mount_1_pitch) $(arg nic_card_mount_1_yaw)"/>
+    <xacro:nic_card_mount prefix="nic_card_mount_1" pose="${-0.081418 + $(arg nic_card_mount_1_translation)} -0.1345 0.012 $(arg nic_card_mount_1_roll) $(arg nic_card_mount_1_pitch) $(arg nic_card_mount_1_yaw)"/>
     <gazebo>
       <joint name="nic_card_mount_1_joint" type="fixed">
@@ -196,5 +196,5 @@
   <!-- NIC Card Mount 2 (center) -->
   <xacro:if value="$(arg nic_card_mount_2_present)">
-    <xacro:nic_card_mount prefix="nic_card_mount_2" pose="${-0.081418 + $(arg nic_card_mount_2_translation)} -0.0945 0.01 $(arg nic_card_mount_2_roll) $(arg nic_card_mount_2_pitch) $(arg nic_card_mount_2_yaw)"/>
+    <xacro:nic_card_mount prefix="nic_card_mount_2" pose="${-0.081418 + $(arg nic_card_mount_2_translation)} -0.0945 0.012 $(arg nic_card_mount_2_roll) $(arg nic_card_mount_2_pitch) $(arg nic_card_mount_2_yaw)"/>
     <gazebo>
       <joint name="nic_card_mount_2_joint" type="fixed">
@@ -206,5 +206,5 @@
   <!-- NIC Card Mount 3 -->
   <xacro:if value="$(arg nic_card_mount_3_present)">
-    <xacro:nic_card_mount prefix="nic_card_mount_3" pose="${-0.081418 + $(arg nic_card_mount_3_translation)} -0.0545 0.01 $(arg nic_card_mount_3_roll) $(arg nic_card_mount_3_pitch) $(arg nic_card_mount_3_yaw)"/>
+    <xacro:nic_card_mount prefix="nic_card_mount_3" pose="${-0.081418 + $(arg nic_card_mount_3_translation)} -0.0545 0.012 $(arg nic_card_mount_3_roll) $(arg nic_card_mount_3_pitch) $(arg nic_card_mount_3_yaw)"/>
     <gazebo>
       <joint name="nic_card_mount_3_joint" type="fixed">
@@ -216,5 +216,5 @@
   <!-- NIC Card Mount 4 (right-most) -->
   <xacro:if value="$(arg nic_card_mount_4_present)">
-    <xacro:nic_card_mount prefix="nic_card_mount_4" pose="${-0.081418 + $(arg nic_card_mount_4_translation)} -0.0145 0.01 $(arg nic_card_mount_4_roll) $(arg nic_card_mount_4_pitch) $(arg nic_card_mount_4_yaw)"/>
+    <xacro:nic_card_mount prefix="nic_card_mount_4" pose="${-0.081418 + $(arg nic_card_mount_4_translation)} -0.0145 0.012 $(arg nic_card_mount_4_roll) $(arg nic_card_mount_4_pitch) $(arg nic_card_mount_4_yaw)"/>
     <gazebo>
       <joint name="nic_card_mount_4_joint" type="fixed">

Commit message: Support up to 3 SC ports per rail (6 total) with min-buffer enforcement

File: aic_description/urdf/task_board.urdf.xacro (robot description, xacro)
@@ -63,4 +63,28 @@
   <xacro:arg name="sc_port_1_pitch" default="0.0"/>
   <xacro:arg name="sc_port_1_yaw" default="0.0"/>
+  <!-- SC Port 2 (SC_RAIL_0) -->
+  <xacro:arg name="sc_port_2_present" default="false"/>
+  <xacro:arg name="sc_port_2_translation" default="0.0"/>
+  <xacro:arg name="sc_port_2_roll" default="0.0"/>
+  <xacro:arg name="sc_port_2_pitch" default="0.0"/>
+  <xacro:arg name="sc_port_2_yaw" default="0.0"/>
+  <!-- SC Port 3 (SC_RAIL_1) -->
+  <xacro:arg name="sc_port_3_present" default="false"/>
+  <xacro:arg name="sc_port_3_translation" default="0.0"/>
+  <xacro:arg name="sc_port_3_roll" default="0.0"/>
+  <xacro:arg name="sc_port_3_pitch" default="0.0"/>
+  <xacro:arg name="sc_port_3_yaw" default="0.0"/>
+  <!-- SC Port 4 (SC_RAIL_1) -->
+  <xacro:arg name="sc_port_4_present" default="false"/>
+  <xacro:arg name="sc_port_4_translation" default="0.0"/>
+  <xacro:arg name="sc_port_4_roll" default="0.0"/>
+  <xacro:arg name="sc_port_4_pitch" default="0.0"/>
+  <xacro:arg name="sc_port_4_yaw" default="0.0"/>
+  <!-- SC Port 5 (SC_RAIL_1) -->
+  <xacro:arg name="sc_port_5_present" default="false"/>
+  <xacro:arg name="sc_port_5_translation" default="0.0"/>
+  <xacro:arg name="sc_port_5_roll" default="0.0"/>
+  <xacro:arg name="sc_port_5_pitch" default="0.0"/>
+  <xacro:arg name="sc_port_5_yaw" default="0.0"/>
   <!-- NIC Card Mount 0 -->
   <xacro:arg name="nic_card_mount_0_present" default="false"/>
@@ -164,11 +188,51 @@
     </gazebo>
   </xacro:if>
-  <!-- SC Port 1 -->
+  <!-- SC Port 1 (SC_RAIL_0, Y=0.0295) -->
   <xacro:if value="$(arg sc_port_1_present)">
-    <xacro:sc_port prefix="sc_port_1" pose="${-0.075 + $(arg sc_port_1_translation)} 0.0705 0.0165 ${1.57 + $(arg sc_port_1_roll)} $(arg sc_port_1_pitch) ${1.57 + $(arg sc_port_1_yaw)}"/>
+    <xacro:sc_port prefix="sc_port_1" pose="${-0.075 + $(arg sc_port_1_translation)} 0.0295 0.0165 ${1.57 + $(arg sc_port_1_roll)} $(arg sc_port_1_pitch) ${1.57 + $(arg sc_port_1_yaw)}"/>
     <gazebo>
       <joint name="sc_port_1_joint" type="fixed">
         <parent>task_board_base_link</parent>
         <child>sc_port_1::sc_port_link</child>
+      </joint>
+    </gazebo>
+  </xacro:if>
+  <!-- SC Port 2 (SC_RAIL_0, Y=0.0295) -->
+  <xacro:if value="$(arg sc_port_2_present)">
+    <xacro:sc_port prefix="sc_port_2" pose="${-0.075 + $(arg sc_port_2_translation)} 0.0295 0.0165 ${1.57 + $(arg sc_port_2_roll)} $(arg sc_port_2_pitch) ${1.57 + $(arg sc_port_2_yaw)}"/>
+    <gazebo>
+      <joint name="sc_port_2_joint" type="fixed">
+        <parent>task_board_base_link</parent>
+        <child>sc_port_2::sc_port_link</child>
+      </joint>
+    </gazebo>
+  </xacro:if>
+  <!-- SC Port 3 (SC_RAIL_1, Y=0.0705) -->
+  <xacro:if value="$(arg sc_port_3_present)">
+    <xacro:sc_port prefix="sc_port_3" pose="${-0.075 + $(arg sc_port_3_translation)} 0.0705 0.0165 ${1.57 + $(arg sc_port_3_roll)} $(arg sc_port_3_pitch) ${1.57 + $(arg sc_port_3_yaw)}"/>
+    <gazebo>
+      <joint name="sc_port_3_joint" type="fixed">
+        <parent>task_board_base_link</parent>
+        <child>sc_port_3::sc_port_link</child>
+      </joint>
+    </gazebo>
+  </xacro:if>
+  <!-- SC Port 4 (SC_RAIL_1, Y=0.0705) -->
+  <xacro:if value="$(arg sc_port_4_present)">
+    <xacro:sc_port prefix="sc_port_4" pose="${-0.075 + $(arg sc_port_4_translation)} 0.0705 0.0165 ${1.57 + $(arg sc_port_4_roll)} $(arg sc_port_4_pitch) ${1.57 + $(arg sc_port_4_yaw)}"/>
+    <gazebo>
+      <joint name="sc_port_4_joint" type="fixed">
+        <parent>task_board_base_link</parent>
+        <child>sc_port_4::sc_port_link</child>
+      </joint>
+    </gazebo>
+  </xacro:if>
+  <!-- SC Port 5 (SC_RAIL_1, Y=0.0705) -->
+  <xacro:if value="$(arg sc_port_5_present)">
+    <xacro:sc_port prefix="sc_port_5" pose="${-0.075 + $(arg sc_port_5_translation)} 0.0705 0.0165 ${1.57 + $(arg sc_port_5_roll)} $(arg sc_port_5_pitch) ${1.57 + $(arg sc_port_5_yaw)}"/>
+    <gazebo>
+      <joint name="sc_port_5_joint" type="fixed">
+        <parent>task_board_base_link</parent>
+        <child>sc_port_5::sc_port_link</child>
       </joint>
     </gazebo>

Commit message: Only modify task_board.urdf.xacro and launch file, revert changes to aic_engine

File: aic_description/urdf/task_board.urdf.xacro (robot description, xacro)
@@ -81,10 +81,4 @@
   <xacro:arg name="sc_port_4_pitch" default="0.0"/>
   <xacro:arg name="sc_port_4_yaw" default="0.0"/>
-  <!-- SC Port 5 (SC_RAIL_1) -->
-  <xacro:arg name="sc_port_5_present" default="false"/>
-  <xacro:arg name="sc_port_5_translation" default="0.0"/>
-  <xacro:arg name="sc_port_5_roll" default="0.0"/>
-  <xacro:arg name="sc_port_5_pitch" default="0.0"/>
-  <xacro:arg name="sc_port_5_yaw" default="0.0"/>
   <!-- NIC Card Mount 0 -->
   <xacro:arg name="nic_card_mount_0_present" default="false"/>
@@ -178,5 +172,5 @@
     </joint>
   </xacro:if>
-  <!-- SC Port 0 -->
+  <!-- SC Port 0 (SC_RAIL_0, Y=0.0295) -->
   <xacro:if value="$(arg sc_port_0_present)">
     <xacro:sc_port prefix="sc_port_0" pose="${-0.075 + $(arg sc_port_0_translation)} 0.0295 0.0165 ${1.57 + $(arg sc_port_0_roll)} $(arg sc_port_0_pitch) ${1.57 + $(arg sc_port_0_yaw)}"/>
@@ -225,14 +219,4 @@
         <parent>task_board_base_link</parent>
         <child>sc_port_4::sc_port_link</child>
-      </joint>
-    </gazebo>
-  </xacro:if>
-  <!-- SC Port 5 (SC_RAIL_1, Y=0.0705) -->
-  <xacro:if value="$(arg sc_port_5_present)">
-    <xacro:sc_port prefix="sc_port_5" pose="${-0.075 + $(arg sc_port_5_translation)} 0.0705 0.0165 ${1.57 + $(arg sc_port_5_roll)} $(arg sc_port_5_pitch) ${1.57 + $(arg sc_port_5_yaw)}"/>
-    <gazebo>
-      <joint name="sc_port_5_joint" type="fixed">
-        <parent>task_board_base_link</parent>
-        <child>sc_port_5::sc_port_link</child>
       </joint>
     </gazebo>

Commit message: Add five mounts

File: aic_description/urdf/task_board.urdf.xacro (robot description, xacro)
@@ -51,4 +51,40 @@
   <xacro:arg name="sc_mount_rail_1_pitch" default="0.0"/>
   <xacro:arg name="sc_mount_rail_1_yaw" default="0.0"/>
+  <!-- SFP Mount Rail 2: X=0.0535, Y=-0.15625 -->
+  <xacro:arg name="sfp_mount_rail_2_present" default="false"/>
+  <xacro:arg name="sfp_mount_rail_2_translation" default="0.0"/>
+  <xacro:arg name="sfp_mount_rail_2_roll" default="0.0"/>
+  <xacro:arg name="sfp_mount_rail_2_pitch" default="0.0"/>
+  <xacro:arg name="sfp_mount_rail_2_yaw" default="0.0"/>
+  <!-- SC Mount Rail 2: X=0.0985, Y=-0.15625 -->
+  <xacro:arg name="sc_mount_rail_2_present" default="false"/>
+  <xacro:arg name="sc_mount_rail_2_translation" default="0.0"/>
+  <xacro:arg name="sc_mount_rail_2_roll" default="0.0"/>
+  <xacro:arg name="sc_mount_rail_2_pitch" default="0.0"/>
+  <xacro:arg name="sc_mount_rail_2_yaw" default="0.0"/>
+  <!-- SFP Mount Rail 3: X=0.0535, Y=-0.05625 -->
+  <xacro:arg name="sfp_mount_rail_3_present" default="false"/>
+  <xacro:arg name="sfp_mount_rail_3_translation" default="0.0"/>
+  <xacro:arg name="sfp_mount_rail_3_roll" default="0.0"/>
+  <xacro:arg name="sfp_mount_rail_3_pitch" default="0.0"/>
+  <xacro:arg name="sfp_mount_rail_3_yaw" default="0.0"/>
+  <!-- SC Mount Rail 3: X=0.0985, Y=-0.05625 -->
+  <xacro:arg name="sc_mount_rail_3_present" default="false"/>
+  <xacro:arg name="sc_mount_rail_3_translation" default="0.0"/>
+  <xacro:arg name="sc_mount_rail_3_roll" default="0.0"/>
+  <xacro:arg name="sc_mount_rail_3_pitch" default="0.0"/>
+  <xacro:arg name="sc_mount_rail_3_yaw" default="0.0"/>
+  <!-- SFP Mount Rail 4: X=0.0535, Y=0.15625 -->
+  <xacro:arg name="sfp_mount_rail_4_present" default="false"/>
+  <xacro:arg name="sfp_mount_rail_4_translation" default="0.0"/>
+  <xacro:arg name="sfp_mount_rail_4_roll" default="0.0"/>
+  <xacro:arg name="sfp_mount_rail_4_pitch" default="0.0"/>
+  <xacro:arg name="sfp_mount_rail_4_yaw" default="0.0"/>
+  <!-- SC Mount Rail 4: X=0.0985, Y=0.15625 -->
+  <xacro:arg name="sc_mount_rail_4_present" default="false"/>
+  <xacro:arg name="sc_mount_rail_4_translation" default="0.0"/>
+  <xacro:arg name="sc_mount_rail_4_roll" default="0.0"/>
+  <xacro:arg name="sc_mount_rail_4_pitch" default="0.0"/>
+  <xacro:arg name="sc_mount_rail_4_yaw" default="0.0"/>
   <!-- SC Port 0 -->
   <xacro:arg name="sc_port_0_present" default="false"/>
@@ -133,5 +169,5 @@
       <parent link="task_board_base_link"/>
       <child link="sfp_mount_rail_0_link"/>
-      <origin xyz="0.055 ${-0.10625 + $(arg sfp_mount_rail_0_translation)} 0.01" rpy="$(arg sfp_mount_rail_0_roll) $(arg sfp_mount_rail_0_pitch) $(arg sfp_mount_rail_0_yaw)"/>
+      <origin xyz="0.055 ${-0.10625 + $(arg sfp_mount_rail_0_translation)} 0.012" rpy="$(arg sfp_mount_rail_0_roll) $(arg sfp_mount_rail_0_pitch) $(arg sfp_mount_rail_0_yaw)"/>
     </joint>
   </xacro:if>
@@ -160,5 +196,5 @@
       <parent link="task_board_base_link"/>
       <child link="sfp_mount_rail_1_link"/>
-      <origin xyz="0.055 ${0.10625 + $(arg sfp_mount_rail_1_translation)} 0.01" rpy="$(arg sfp_mount_rail_1_roll) $(arg sfp_mount_rail_1_pitch) $(arg sfp_mount_rail_1_yaw)"/>
+      <origin xyz="0.055 ${0.10625 + $(arg sfp_mount_rail_1_translation)} 0.012" rpy="$(arg sfp_mount_rail_1_roll) $(arg sfp_mount_rail_1_pitch) $(arg sfp_mount_rail_1_yaw)"/>
     </joint>
   </xacro:if>
@@ -169,5 +205,59 @@
       <parent link="task_board_base_link"/>
       <child link="sc_mount_rail_1_link"/>
-      <origin xyz="0.0985 ${0.10625 + $(arg sc_mount_rail_1_translation)} 0.01" rpy="$(arg sc_mount_rail_1_roll) $(arg sc_mount_rail_1_pitch) $(arg sc_mount_rail_1_yaw)"/>
+      <origin xyz="0.0985 ${0.10625 + $(arg sc_mount_rail_1_translation)} 0.012" rpy="$(arg sc_mount_rail_1_roll) $(arg sc_mount_rail_1_pitch) $(arg sc_mount_rail_1_yaw)"/>
+    </joint>
+  </xacro:if>
+  <!-- SFP Mount Rail 2: X=0.055, Y=-0.15625 -->
+  <xacro:if value="$(arg sfp_mount_rail_2_present)">
+    <xacro:sfp_mount prefix="sfp_mount_rail_2_"/>
+    <joint name="sfp_mount_rail_2_joint" type="fixed">
+      <parent link="task_board_base_link"/>
+      <child link="sfp_mount_rail_2_link"/>
+      <origin xyz="0.055 ${-0.15625 + $(arg sfp_mount_rail_2_translation)} 0.012" rpy="$(arg sfp_mount_rail_2_roll) $(arg sfp_mount_rail_2_pitch) $(arg sfp_mount_rail_2_yaw)"/>
+    </joint>
+  </xacro:if>
+  <!-- SC Mount Rail 2: X=0.1, Y=-0.15625 -->
+  <xacro:if value="$(arg sc_mount_rail_2_present)">
+    <xacro:sc_mount prefix="sc_mount_rail_2_"/>
+    <joint name="sc_mount_rail_2_joint" type="fixed">
+      <parent link="task_board_base_link"/>
+      <child link="sc_mount_rail_2_link"/>
+      <origin xyz="0.1 ${-0.15625 + $(arg sc_mount_rail_2_translation)} 0.012" rpy="$(arg sc_mount_rail_2_roll) $(arg sc_mount_rail_2_pitch) $(arg sc_mount_rail_2_yaw)"/>
+    </joint>
+  </xacro:if>
+  <!-- SFP Mount Rail 3: X=0.055, Y=-0.05625 -->
+  <xacro:if value="$(arg sfp_mount_rail_3_present)">
+    <xacro:sfp_mount prefix="sfp_mount_rail_3_"/>
+    <joint name="sfp_mount_rail_3_joint" type="fixed">
+      <parent link="task_board_base_link"/>
+      <child link="sfp_mount_rail_3_link"/>
+      <origin xyz="0.055 ${-0.05625 + $(arg sfp_mount_rail_3_translation)} 0.012" rpy="$(arg sfp_mount_rail_3_roll) $(arg sfp_mount_rail_3_pitch) $(arg sfp_mount_rail_3_yaw)"/>
+    </joint>
+  </xacro:if>
+  <!-- SC Mount Rail 3: X=0.1, Y=-0.05625 -->
+  <xacro:if value="$(arg sc_mount_rail_3_present)">
+    <xacro:sc_mount prefix="sc_mount_rail_3_"/>
+    <joint name="sc_mount_rail_3_joint" type="fixed">
+      <parent link="task_board_base_link"/>
+      <child link="sc_mount_rail_3_link"/>
+      <origin xyz="0.1 ${-0.05625 + $(arg sc_mount_rail_3_translation)} 0.012" rpy="$(arg sc_mount_rail_3_roll) $(arg sc_mount_rail_3_pitch) $(arg sc_mount_rail_3_yaw)"/>
+    </joint>
+  </xacro:if>
+  <!-- SFP Mount Rail 4: X=0.055, Y=0.15625 -->
+  <xacro:if value="$(arg sfp_mount_rail_4_present)">
+    <xacro:sfp_mount prefix="sfp_mount_rail_4_"/>
+    <joint name="sfp_mount_rail_4_joint" type="fixed">
+      <parent link="task_board_base_link"/>
+      <child link="sfp_mount_rail_4_link"/>
+      <origin xyz="0.055 ${0.15625 + $(arg sfp_mount_rail_4_translation)} 0.012" rpy="$(arg sfp_mount_rail_4_roll) $(arg sfp_mount_rail_4_pitch) $(arg sfp_mount_rail_4_yaw)"/>
+    </joint>
+  </xacro:if>
+  <!-- SC Mount Rail 4: X=0.0985, Y=0.15625 -->
+  <xacro:if value="$(arg sc_mount_rail_4_present)">
+    <xacro:sc_mount prefix="sc_mount_rail_4_"/>
+    <joint name="sc_mount_rail_4_joint" type="fixed">
+      <parent link="task_board_base_link"/>
+      <child link="sc_mount_rail_4_link"/>
+      <origin xyz="0.0985 ${0.15625 + $(arg sc_mount_rail_4_translation)} 0.012" rpy="$(arg sc_mount_rail_4_roll) $(arg sc_mount_rail_4_pitch) $(arg sc_mount_rail_4_yaw)"/>
     </joint>
   </xacro:if>
