Commit message: Remove mimic joint for gripper right finger
Signed-off-by: Yadunund <yadunund@intrinsic.ai>

File: aic_utils/aic_mujoco/config/mujoco_ros2_control.xacro (robot description, xacro)
@@ -46,14 +46,4 @@
       </state_interface>
     </joint>
-    <joint name="$(arg gripper_tf_prefix)right_finger_joint">
-      <param name="mimic">$(arg gripper_tf_prefix)left_finger_joint</param>
-      <param name="multiplier">1</param>
-      <state_interface name="position">
-        <param name="initial_value">$(arg gripper_initial_pos)</param>
-      </state_interface>
-      <state_interface name="velocity">
-        <param name="initial_value">0.0</param>
-      </state_interface>
-    </joint>
   </ros2_control>
 </robot>
