Commit message: Tweak xacro mount collisions
Signed-off-by: Ian Chen <iche@intrinsic.ai>

File: aic_assets/models/SC Mount/sc_mount_macro.xacro (robot description, xacro)
@@ -53,5 +53,5 @@
         <origin xyz="0.017774 0.0 0.008656" rpy="0.0 0.785398 0.0"/>
         <geometry>
-          <box size="0.025812 0.014 0.001239"/>
+          <box size="0.009 0.014 0.001239"/>
         </geometry>
       </collision>

File: aic_assets/models/SFP Mount/sfp_mount_macro.xacro (robot description, xacro)
@@ -33,13 +33,13 @@
       </collision>
       <collision name="iso_4762_m2_x_8072_collider_box_003">
-        <origin xyz="0.021242 0.007723 0.013979" rpy="0.0 -0.785398 0.0"/>
+        <origin xyz="0.021242 0.0080 0.013979" rpy="0.0 -0.785398 0.0"/>
         <geometry>
-          <box size="0.036111 0.002305 0.010956"/>
+          <box size="0.036111 0.0018 0.010956"/>
         </geometry>
       </collision>
       <collision name="iso_4762_m2_x_8072_collider_box_004">
-        <origin xyz="0.021003 -0.007938 0.014217" rpy="0.0 -0.785398 0.0"/>
+        <origin xyz="0.021003 -0.008 0.014217" rpy="0.0 -0.785398 0.0"/>
         <geometry>
-          <box size="0.036111 0.001875 0.01163"/>
+          <box size="0.036111 0.0018 0.01163"/>
         </geometry>
       </collision>

Commit message: reduce mount collisions
Signed-off-by: Ian Chen <iche@intrinsic.ai>

File: aic_assets/models/SC Mount/sc_mount_macro.xacro (robot description, xacro)
@@ -23,5 +23,5 @@
         <origin xyz="0.022568 -0.0054 0.013451" rpy="0.0 0.785398 0.0"/>
         <geometry>
-          <box size="0.025812 0.0032 0.013799"/>
+          <box size="0.025812 0.0022 0.013799"/>
         </geometry>
       </collision>
@@ -29,5 +29,5 @@
         <origin xyz="0.022568 0.00585 0.013451" rpy="0.0 0.785398 0.0"/>
         <geometry>
-          <box size="0.025812 0.0023 0.013799"/>
+          <box size="0.025812 0.0022 0.013799"/>
         </geometry>
       </collision>
@@ -35,5 +35,5 @@
         <origin xyz="0.01415 0.0 0.02187" rpy="0.0 0.785398 0.0"/>
         <geometry>
-          <box size="0.002 0.014 0.013799"/>
+          <box size="0.0012 0.014 0.013799"/>
         </geometry>
       </collision>
@@ -41,5 +41,5 @@
         <origin xyz="0.031064 0.0 0.004956" rpy="0.0 0.785398 0.0"/>
         <geometry>
-          <box size="0.001842 0.014 0.013799"/>
+          <box size="0.001042 0.014 0.013799"/>
         </geometry>
       </collision>

File: aic_assets/models/SFP Mount/sfp_mount_macro.xacro (robot description, xacro)
@@ -23,5 +23,5 @@
         <origin xyz="0.016366 0.0 0.017144" rpy="0.0 -0.785398 0.0"/>
         <geometry>
-          <box size="0.038533 0.01775 0.001728"/>
+          <box size="0.038533 0.01775 0.001028"/>
         </geometry>
       </collision>
@@ -29,5 +29,5 @@
         <origin xyz="0.028636 0.0 0.012684" rpy="0.0 -0.785398 0.0"/>
         <geometry>
-          <box size="0.027485 0.01775 0.003688"/>
+          <box size="0.027485 0.01775 0.002888"/>
         </geometry>
       </collision>
@@ -35,5 +35,5 @@
         <origin xyz="0.021242 0.007723 0.013979" rpy="0.0 -0.785398 0.0"/>
         <geometry>
-          <box size="0.036111 0.002305 0.010956"/>
+          <box size="0.036111 0.0012 0.010956"/>
         </geometry>
       </collision>
@@ -41,5 +41,5 @@
         <origin xyz="0.021003 -0.007938 0.014217" rpy="0.0 -0.785398 0.0"/>
         <geometry>
-          <box size="0.036111 0.001875 0.01163"/>
+          <box size="0.036111 0.0012 0.01163"/>
         </geometry>
       </collision>

Commit message: reduce mount collisions (#533)
Signed-off-by: Ian Chen <iche@intrinsic.ai>
Co-authored-by: Luca Della Vedova <lucadv@intrinsic.ai>

File: aic_assets/models/SC Mount/sc_mount_macro.xacro (robot description, xacro)
@@ -23,5 +23,5 @@
         <origin xyz="0.022568 -0.0054 0.013451" rpy="0.0 0.785398 0.0"/>
         <geometry>
-          <box size="0.025812 0.0032 0.013799"/>
+          <box size="0.025812 0.0022 0.013799"/>
         </geometry>
       </collision>
@@ -29,5 +29,5 @@
         <origin xyz="0.022568 0.00585 0.013451" rpy="0.0 0.785398 0.0"/>
         <geometry>
-          <box size="0.025812 0.0023 0.013799"/>
+          <box size="0.025812 0.0022 0.013799"/>
         </geometry>
       </collision>
@@ -35,5 +35,5 @@
         <origin xyz="0.01415 0.0 0.02187" rpy="0.0 0.785398 0.0"/>
         <geometry>
-          <box size="0.002 0.014 0.013799"/>
+          <box size="0.0012 0.014 0.013799"/>
         </geometry>
       </collision>
@@ -41,5 +41,5 @@
         <origin xyz="0.031064 0.0 0.004956" rpy="0.0 0.785398 0.0"/>
         <geometry>
-          <box size="0.001842 0.014 0.013799"/>
+          <box size="0.001042 0.014 0.013799"/>
         </geometry>
       </collision>

File: aic_assets/models/SFP Mount/sfp_mount_macro.xacro (robot description, xacro)
@@ -23,5 +23,5 @@
         <origin xyz="0.016366 0.0 0.017144" rpy="0.0 -0.785398 0.0"/>
         <geometry>
-          <box size="0.038533 0.01775 0.001728"/>
+          <box size="0.038533 0.01775 0.001028"/>
         </geometry>
       </collision>
@@ -29,5 +29,5 @@
         <origin xyz="0.028636 0.0 0.012684" rpy="0.0 -0.785398 0.0"/>
         <geometry>
-          <box size="0.027485 0.01775 0.003688"/>
+          <box size="0.027485 0.01775 0.002888"/>
         </geometry>
       </collision>
@@ -35,5 +35,5 @@
         <origin xyz="0.021242 0.0080 0.013979" rpy="0.0 -0.785398 0.0"/>
         <geometry>
-          <box size="0.036111 0.0018 0.010956"/>
+          <box size="0.036111 0.0012 0.010956"/>
         </geometry>
       </collision>
@@ -41,5 +41,5 @@
         <origin xyz="0.021003 -0.008 0.014217" rpy="0.0 -0.785398 0.0"/>
         <geometry>
-          <box size="0.036111 0.0018 0.01163"/>
+          <box size="0.036111 0.0012 0.01163"/>
         </geometry>
       </collision>
