Commit message: replace sfp and nic card mount urdf with gazebo include tag
Signed-off-by: Ian Chen <ichen@openrobotics.org>

File: aic_assets/models/NIC Card Mount/nic_card_mount_macro.xacro (robot description, xacro)
@@ -1,189 +1,12 @@
 <?xml version="1.0" ?>
 <robot xmlns:xacro="http://wiki.ros.org/xacro">
-  <xacro:macro name="nic_card_mount" params="prefix">
-    <!-- NIC Card Mount Link -->
-    <link name="${prefix}link">
-      <inertial>
-        <origin xyz="0 0 0" rpy="0 0 0"/>
-        <mass value="0.1"/>
-        <inertia ixx="0.001" ixy="0.0" ixz="0.0" iyy="0.001" iyz="0.0" izz="0.001"/>
-      </inertial>
-      <visual name="nic_card_mount_visual">
-        <origin xyz="0 0 0" rpy="0 0 0"/>
-        <geometry>
-          <mesh filename="package://aic_assets/models/NIC Card Mount/nic_card_mount_visual.glb"/>
-        </geometry>
-      </visual>
-      <collision name="v1015085006_collider_box">
-        <origin xyz="0.007 -0.0255 0.0775" rpy="0.0 0.0 1.570796"/>
-        <geometry>
-          <box size="0.005 0.072 0.155"/>
-        </geometry>
-      </collision>
-      <collision name="v1015085006_collider_box_001">
-        <origin xyz="-0.048467 -0.0155 0.162" rpy="0.0 0.0 1.570796"/>
-        <geometry>
-          <box size="0.025 0.039374 0.014"/>
-        </geometry>
-      </collision>
-      <collision name="v1015085006_collider_box_002">
-        <origin xyz="0.0405 -0.01425 0.1055" rpy="0.0 0.0 1.570796"/>
-        <geometry>
-          <box size="0.0275 0.005 0.103"/>
-        </geometry>
-      </collision>
-      <collision name="v1015085006_collider_box_003">
-        <origin xyz="0.0 -0.0125 0.0055" rpy="0.0 0.0 1.570796"/>
-        <geometry>
-          <box size="0.031 0.058 0.011"/>
-        </geometry>
-      </collision>
-      <collision name="v1015085006_collider_box004_collider_box">
-        <origin xyz="-0.045132 -0.0255 0.137803" rpy="0.0 0.0 1.570796"/>
-        <geometry>
-          <box size="0.005 0.036343 0.034395"/>
-        </geometry>
-      </collision>
-    </link>
-    <!-- NIC Card Link -->
-    <link name="${prefix}card_link">
-      <inertial>
-        <origin xyz="0 0 0" rpy="0 0 0"/>
-        <mass value="0.15"/>
-        <inertia ixx="0.001" ixy="0.0" ixz="0.0" iyy="0.001" iyz="0.0" izz="0.001"/>
-      </inertial>
-      <visual name="nic_card_visual">
-        <origin xyz="0 0 0" rpy="0 0 0"/>
-        <geometry>
-          <mesh filename="package://aic_assets/models/NIC Card Mount/nic_card_visual.glb"/>
-        </geometry>
-      </visual>
-      <collision name="pcb_collider_box">
-        <origin xyz="0.0 0.0 -0.0008" rpy="0.0 0.0 0.0"/>
-        <geometry>
-          <box size="0.056 0.145 0.0016"/>
-        </geometry>
-      </collision>
-      <collision name="pcb_collider_box_001">
-        <origin xyz="0.0065 -0.0025 -0.0008" rpy="0.0 0.0 0.0"/>
-        <geometry>
-          <box size="0.069 0.051 0.0016"/>
-        </geometry>
-      </collision>
-      <collision name="pcb_collider_box_002">
-        <origin xyz="0.004 -0.02475 -0.0008" rpy="0.0 0.0 0.0"/>
-        <geometry>
-          <box size="0.064 0.0955 0.0016"/>
-        </geometry>
-      </collision>
-      <collision name="cube001_collider_box">
-        <origin xyz="0.025006 -0.00041 0.00575" rpy="0.0 0.0 0.0"/>
-        <geometry>
-          <box size="0.004 0.14 0.0115"/>
-        </geometry>
-      </collision>
-      <collision name="cube001_collider_box_001">
-        <origin xyz="-0.0029 -0.0015 0.008" rpy="0.0 0.0 0.0"/>
-        <geometry>
-          <box size="0.047 0.052 0.011"/>
-        </geometry>
-      </collision>
-      <collision name="cube001_collider_box_002">
-        <origin xyz="-0.0029 -0.0015 0.001228" rpy="0.0 0.0 0.0"/>
-        <geometry>
-          <box size="0.043 0.048 0.003149"/>
-        </geometry>
-      </collision>
-      <collision name="10099100-011lfc001_collider_box">
-        <origin xyz="-0.017799 -0.052954 0.00548" rpy="3.128092 0.0 0.0"/>
-        <geometry>
-          <box size="0.001099 0.04872 0.011083"/>
-        </geometry>
-      </collision>
-      <collision name="10099100-011lfc001_collider_box.001">
-        <origin xyz="-0.002687 -0.052954 0.005461" rpy="3.128092 0.0 0.0"/>
-        <geometry>
-          <box size="0.001125 0.04872 0.011121"/>
-        </geometry>
-      </collision>
-      <collision name="10099100-011lfc001_collider_box.002">
-        <origin xyz="-0.010237 -0.052889 0.010234" rpy="3.128092 0.0 0.0"/>
-        <geometry>
-          <box size="0.016224 0.04872 0.000923"/>
-        </geometry>
-      </collision>
-      <collision name="10099100-011lfc001_collider_box.003">
-        <origin xyz="-0.010237 -0.053024 0.000296" rpy="3.128092 0.0 0.0"/>
-        <geometry>
-          <box size="0.016224 0.04872 0.001054"/>
-        </geometry>
-      </collision>
-      <collision name="10099100-011lfc001_collider_box.004">
-        <origin xyz="-0.010237 -0.028738 0.003845" rpy="3.128092 0.0 0.0"/>
-        <geometry>
-          <box size="0.016224 0.00025 0.013698"/>
-        </geometry>
-      </collision>
-      <collision name="10099100-011lfc001_collider_box.005">
-        <origin xyz="0.005401 -0.052954 0.00548" rpy="3.128092 0.0 0.0"/>
-        <geometry>
-          <box size="0.001099 0.04872 0.011083"/>
-        </geometry>
-      </collision>
-      <collision name="10099100-011lfc001_collider_box.006">
-        <origin xyz="0.020513 -0.052954 0.005461" rpy="3.128092 0.0 0.0"/>
-        <geometry>
-          <box size="0.001125 0.04872 0.011121"/>
-        </geometry>
-      </collision>
-      <collision name="10099100-011lfc001_collider_box.007">
-        <origin xyz="0.012963 -0.052889 0.010234" rpy="3.128092 0.0 0.0"/>
-        <geometry>
-          <box size="0.016224 0.04872 0.00092"/>
-        </geometry>
-      </collision>
-      <collision name="10099100-011lfc001_collider_box.008">
-        <origin xyz="0.012963 -0.053024 0.000296" rpy="3.128092 0.0 0.0"/>
-        <geometry>
-          <box size="0.016224 0.04872 0.001054"/>
-        </geometry>
-      </collision>
-      <collision name="10099100-011lfc001_collider_box.009">
-        <origin xyz="0.012963 -0.028738 0.003845" rpy="3.128092 0.0 0.0"/>
-        <geometry>
-          <box size="0.016224 0.00025 0.01369"/>
-        </geometry>
-      </collision>
-      <collision name="plane001_collider_box">
-        <origin xyz="-0.007649 -0.074646 -0.0007515" rpy="0.0 0.0 0.0"/>
-        <geometry>
-          <box size="0.113402 0.000875 0.003449"/>
-        </geometry>
-      </collision>
-      <collision name="plane001_collider_box.001">
-        <origin xyz="-0.007649 -0.074646 0.01352" rpy="0.0 0.0 0.0"/>
-        <geometry>
-          <box size="0.113402 0.000875 0.00501"/>
-        </geometry>
-      </collision>
-      <collision name="plane001_collider_box.002">
-        <origin xyz="0.038559 -0.074646 0.006455" rpy="0.0 0.0 0.0"/>
-        <geometry>
-          <box size="0.036181 0.000875 0.01112"/>
-        </geometry>
-      </collision>
-      <collision name="plane001_collider_box.003">
-        <origin xyz="-0.041261 -0.074646 0.006455" rpy="0.0 0.0 0.0"/>
-        <geometry>
-          <box size="0.046178 0.000875 0.011123"/>
-        </geometry>
-      </collision>
-    </link>
-    <!-- Joint connecting card to mount -->
-    <joint name="${prefix}card_joint" type="fixed">
-      <parent link="${prefix}link"/>
-      <child link="${prefix}card_link"/>
-      <origin xyz="0 -0.01785 0.0799" rpy="-1.57 0 0"/>
-    </joint>
+  <xacro:macro name="nic_card_mount" params="prefix pose">
+    <gazebo>
+      <include>
+        <name>${prefix}</name>
+        <uri>package://aic_assets/models/NIC Card Mount</uri>
+        <pose>${pose}</pose>
+      </include>
+    </gazebo>
   </xacro:macro>
 </robot>

File: aic_assets/models/SC Port/sc_port_macro.xacro (robot description, xacro)
@@ -1,78 +1,12 @@
 <?xml version="1.0" ?>
 <robot xmlns:xacro="http://wiki.ros.org/xacro">
-  <xacro:macro name="sc_port" params="prefix">
-    <link name="${prefix}link">
-      <inertial>
-        <origin xyz="0 0 0" rpy="0 0 0"/>
-        <mass value="0.04"/>
-        <inertia ixx="0.0001" ixy="0.0" ixz="0.0" iyy="0.0001" iyz="0.0" izz="0.0001"/>
-      </inertial>
-      <visual name="sc_port_visual">
-        <origin xyz="0 0 0" rpy="0 0 0"/>
-        <geometry>
-          <mesh filename="package://aic_assets/models/SC Port/sc_port_visual.glb"/>
-        </geometry>
-      </visual>
-      <collision name="cube_collider_box">
-        <origin xyz="0.011922 0.0 0.0" rpy="0.0 0.0 0.0"/>
-        <geometry>
-          <box size="0.001937 0.027432 0.0093"/>
-        </geometry>
-      </collision>
-      <collision name="cube_collider_box_001">
-        <origin xyz="0.0 0.0 0.004225" rpy="0.0 0.0 0.0"/>
-        <geometry>
-          <box size="0.025781 0.0108 0.00085"/>
-        </geometry>
-      </collision>
-      <collision name="cube_collider_box_mid">
-        <origin xyz="0.0 0.0 0.004225" rpy="0.0 0.0 0.0"/>
-        <geometry>
-          <box size="0.0103 0.027432 0.00085"/>
-        </geometry>
-      </collision>
-      <collision name="cube_collider_box_mid02">
-        <origin xyz="0.01 0.0 0.004225" rpy="0.0 0.0 0.0"/>
-        <geometry>
-          <box size="0.005 0.027432 0.00085"/>
-        </geometry>
-      </collision>
-      <collision name="cube_collider_box_mid03">
-        <origin xyz="-0.01 0.0 0.004225" rpy="0.0 0.0 0.0"/>
-        <geometry>
-          <box size="0.005 0.027432 0.00085"/>
-        </geometry>
-      </collision>
-      <collision name="cube_collider_box_002">
-        <origin xyz="0.0 0.0 -0.004225" rpy="0.0 0.0 0.0"/>
-        <geometry>
-          <box size="0.02565 0.027432 0.00085"/>
-        </geometry>
-      </collision>
-      <collision name="cube_collider_box_003">
-        <origin xyz="-0.011922 0.0 0.0" rpy="0.0 0.0 0.0"/>
-        <geometry>
-          <box size="0.001937 0.027432 0.0093"/>
-        </geometry>
-      </collision>
-      <collision name="cube_collider_box_004">
-        <origin xyz="-0.014683 0.0 0.0" rpy="0.0 0.0 0.0"/>
-        <geometry>
-          <box size="0.005484 0.003048 0.0093"/>
-        </geometry>
-      </collision>
-      <collision name="cube_collider_box_005">
-        <origin xyz="0.014683 0.0 0.0" rpy="0.0 0.0 0.0"/>
-        <geometry>
-          <box size="0.005484 0.003048 0.0093"/>
-        </geometry>
-      </collision>
-      <collision name="cube_collider_box_006">
-        <origin xyz="0.0 0.0 0.0" rpy="0.0 0.0 0.0"/>
-        <geometry>
-          <box size="0.003492 0.027432 0.0093"/>
-        </geometry>
-      </collision>
-    </link>
+  <xacro:macro name="sc_port" params="prefix pose">
+    <gazebo>
+      <include>
+        <name>${prefix}</name>
+        <uri>package://aic_assets/models/SC Port</uri>
+        <pose>${pose}</pose>
+      </include>
+    </gazebo>
   </xacro:macro>
 </robot>

File: aic_description/urdf/task_board.urdf.xacro (robot description, xacro)
@@ -114,52 +114,59 @@
   </joint>
   <!-- SC Port 01 -->
-  <xacro:sc_port prefix="sc_port_01_"/>
-  <joint name="sc_port_01_joint" type="fixed">
-    <parent link="task_board_base_link"/>
-    <child link="sc_port_01_link"/>
-    <origin xyz="${-0.075 + $(arg sc_port_01_delta_x)} ${0.0295 + $(arg sc_port_01_delta_y)} ${0.01 + $(arg sc_port_01_delta_z)}" rpy="1.57 0 1.57"/>
-  </joint>
+  <xacro:sc_port prefix="sc_port_01" pose="${-0.075 + $(arg sc_port_01_delta_x)} ${0.0295 + $(arg sc_port_01_delta_y)} ${0.01 + $(arg sc_port_01_delta_z)} 1.57 0 1.57"/>
+  <gazebo>
+    <joint name="sc_port_01_joint" type="fixed">
+      <parent> task_board_base_link</parent>
+      <child>sc_port_01::sc_port_link</child>
+    </joint>
+  </gazebo>
   <!-- SC Port 02 -->
-  <xacro:sc_port prefix="sc_port_02_"/>
-  <joint name="sc_port_02_joint" type="fixed">
-    <parent link="task_board_base_link"/>
-    <child link="sc_port_02_link"/>
-    <origin xyz="${-0.075 + $(arg sc_port_02_delta_x)} ${0.0705 + $(arg sc_port_02_delta_y)} ${0.01 + $(arg sc_port_02_delta_z)}" rpy="1.57 0 1.57"/>
-  </joint>
+  <xacro:sc_port prefix="sc_port_02" pose="${-0.075 + $(arg sc_port_02_delta_x)} ${0.0705 + $(arg sc_port_02_delta_y)} ${0.01 + $(arg sc_port_02_delta_z)} 1.57 0 1.57"/>
+  <gazebo>
+    <joint name="sc_port_02_joint" type="fixed">
+      <parent> task_board_base_link</parent>
+      <child>sc_port_02::sc_port_link</child>
+    </joint>
+  </gazebo>
   <!-- NIC Card Mount 01 -->
-  <xacro:nic_card_mount prefix="nic_card_mount_01_"/>
-  <joint name="nic_card_mount_01_joint" type="fixed">
-    <parent link="task_board_base_link"/>
-    <child link="nic_card_mount_01_link"/>
-    <origin xyz="${-0.081418 + $(arg nic_card_mount_01_delta_x)} ${-0.0145 + $(arg nic_card_mount_01_delta_y)} ${0.01 + $(arg nic_card_mount_01_delta_z)}" rpy="0 0 0"/>
-  </joint>
+  <xacro:nic_card_mount prefix="nic_card_mount_01" pose="${-0.081418 + $(arg nic_card_mount_01_delta_x)} ${-0.0145 + $(arg nic_card_mount_01_delta_y)} ${0.01 + $(arg nic_card_mount_01_delta_z)} 0 0 0"/>
+  <gazebo>
+    <joint name="nic_card_mount_01_joint" type="fixed">
+      <parent>task_board_base_link</parent>
+      <child>nic_card_mount_01::nic_card_mount_link</child>
+    </joint>
+  </gazebo>
   <!-- NIC Card Mount 02 -->
-  <xacro:nic_card_mount prefix="nic_card_mount_02_"/>
-  <joint name="nic_card_mount_02_joint" type="fixed">
-    <parent link="task_board_base_link"/>
-    <child link="nic_card_mount_02_link"/>
-    <origin xyz="${-0.081418 + $(arg nic_card_mount_02_delta_x)} ${-0.0545 + $(arg nic_card_mount_02_delta_y)} ${0.01 + $(arg nic_card_mount_02_delta_z)}" rpy="0 0 0"/>
-  </joint>
+  <xacro:nic_card_mount prefix="nic_card_mount_02" pose="${-0.081418 + $(arg nic_card_mount_02_delta_x)} ${-0.0545 + $(arg nic_card_mount_02_delta_y)} ${0.01 + $(arg nic_card_mount_02_delta_z)} 0 0 0"/>
+  <gazebo>
+    <joint name="nic_card_mount_02_joint" type="fixed">
+      <parent>task_board_base_link</parent>
+      <child>nic_card_mount_02::nic_card_mount_link</child>
+    </joint>
+  </gazebo>
   <!-- NIC Card Mount 03 -->
-  <xacro:nic_card_mount prefix="nic_card_mount_03_"/>
-  <joint name="nic_card_mount_03_joint" type="fixed">
-    <parent link="task_board_base_link"/>
-    <child link="nic_card_mount_03_link"/>
-    <origin xyz="${-0.081418 + $(arg nic_card_mount_03_delta_x)} ${-0.0945 + $(arg nic_card_mount_03_delta_y)} ${0.01 + $(arg nic_card_mount_03_delta_z)}" rpy="0 0 0"/>
-  </joint>
+  <xacro:nic_card_mount prefix="nic_card_mount_03" pose="${-0.081418 + $(arg nic_card_mount_03_delta_x)} ${-0.0945 + $(arg nic_card_mount_03_delta_y)} ${0.01 + $(arg nic_card_mount_03_delta_z)} 0 0 0"/>
+  <gazebo>
+    <joint name="nic_card_mount_03_joint" type="fixed">
+      <parent>task_board_base_link</parent>
+      <child>nic_card_mount_03::nic_card_mount_link</child>
+    </joint>
+  </gazebo>
   <!-- NIC Card Mount 04 -->
-  <xacro:nic_card_mount prefix="nic_card_mount_04_"/>
-  <joint name="nic_card_mount_04_joint" type="fixed">
-    <parent link="task_board_base_link"/>
-    <child link="nic_card_mount_04_link"/>
-    <origin xyz="${-0.081418 + $(arg nic_card_mount_04_delta_x)} ${-0.1345 + $(arg nic_card_mount_04_delta_y)} ${0.01 + $(arg nic_card_mount_04_delta_z)}" rpy="0 0 0"/>
-  </joint>
+  <xacro:nic_card_mount prefix="nic_card_mount_04" pose="${-0.081418 + $(arg nic_card_mount_04_delta_x)} ${-0.1345 + $(arg nic_card_mount_04_delta_y)} ${0.01 + $(arg nic_card_mount_04_delta_z)} 0 0 0"/>
+  <gazebo>
+    <joint name="nic_card_mount_04_joint" type="fixed">
+      <parent>task_board_base_link</parent>
+      <child>nic_card_mount_04::nic_card_mount_link</child>
+    </joint>
+  </gazebo>
   <!-- NIC Card Mount 05 -->
-  <xacro:nic_card_mount prefix="nic_card_mount_05_"/>
-  <joint name="nic_card_mount_05_joint" type="fixed">
-    <parent link="task_board_base_link"/>
-    <child link="nic_card_mount_05_link"/>
-    <origin xyz="${-0.081418 + $(arg nic_card_mount_05_delta_x)} ${-0.1745 + $(arg nic_card_mount_05_delta_y)} ${0.01 + $(arg nic_card_mount_05_delta_z)}" rpy="0 0 0"/>
-  </joint>
+  <xacro:nic_card_mount prefix="nic_card_mount_05" pose="${-0.081418 + $(arg nic_card_mount_05_delta_x)} ${-0.1745 + $(arg nic_card_mount_05_delta_y)} ${0.01 + $(arg nic_card_mount_05_delta_z)} 0 0 0"/>
+  <gazebo>
+    <joint name="nic_card_mount_05_joint" type="fixed">
+      <parent>task_board_base_link</parent>
+      <child>nic_card_mount_05::nic_card_mount_link</child>
+    </joint>
+  </gazebo>
   <gazebo>
     <static>true</static>

Commit message: WIP Adding plugins to standalone models
Signed-off-by: Luca Della Vedova <lucadv@intrinsic.ai>

File: aic_assets/models/NIC Card Mount/nic_card_mount_macro.xacro (robot description, xacro)
@@ -7,22 +7,4 @@
         <uri>package://aic_assets/models/NIC Card Mount</uri>
         <pose>${pose}</pose>
-        <plugin
-          filename="gz-sim-touchplugin-system"
-          name="gz::sim::systems::TouchPlugin">
-          <target>sfp_tip_link/collision/contact_collision</target>
-          <time>1</time>
-          <namespace>${prefix}/sfp_port_0</namespace>
-          <enabled>true</enabled>
-          <collision>contact_collision_01</collision>
-        </plugin>
-        <plugin
-          filename="gz-sim-touchplugin-system"
-          name="gz::sim::systems::TouchPlugin">
-          <target>sfp_tip_link/collision/contact_collision</target>
-          <time>1</time>
-          <namespace>${prefix}/sfp_port_1</namespace>
-          <enabled>true</enabled>
-          <collision>contact_collision_02</collision>
-        </plugin>
       </include>
     </gazebo>

File: aic_assets/models/SC Port/sc_port_macro.xacro (robot description, xacro)
@@ -7,12 +7,4 @@
         <uri>package://aic_assets/models/SC Port</uri>
         <pose>${pose}</pose>
-        <plugin
-          filename="gz-sim-touchplugin-system"
-          name="gz::sim::systems::TouchPlugin">
-          <target>sc_plug</target>
-          <time>1</time>
-          <namespace>${prefix}/sc_port_base</namespace>
-          <enabled>true</enabled>
-        </plugin>
       </include>
     </gazebo>

Commit message: Revert changes to existing models
Signed-off-by: Luca Della Vedova <lucadv@intrinsic.ai>

File: aic_assets/models/NIC Card Mount/nic_card_mount_macro.xacro (robot description, xacro)
@@ -7,4 +7,22 @@
         <uri>package://aic_assets/models/NIC Card Mount</uri>
         <pose>${pose}</pose>
+        <plugin
+          filename="gz-sim-touchplugin-system"
+          name="gz::sim::systems::TouchPlugin">
+          <target>sfp_tip_link/collision/contact_collision</target>
+          <time>1</time>
+          <namespace>${prefix}/sfp_port_0</namespace>
+          <enabled>true</enabled>
+          <collision>contact_collision_01</collision>
+        </plugin>
+        <plugin
+          filename="gz-sim-touchplugin-system"
+          name="gz::sim::systems::TouchPlugin">
+          <target>sfp_tip_link/collision/contact_collision</target>
+          <time>1</time>
+          <namespace>${prefix}/sfp_port_1</namespace>
+          <enabled>true</enabled>
+          <collision>contact_collision_02</collision>
+        </plugin>
       </include>
     </gazebo>

File: aic_assets/models/SC Port/sc_port_macro.xacro (robot description, xacro)
@@ -7,4 +7,12 @@
         <uri>package://aic_assets/models/SC Port</uri>
         <pose>${pose}</pose>
+        <plugin
+          filename="gz-sim-touchplugin-system"
+          name="gz::sim::systems::TouchPlugin">
+          <target>sc_plug</target>
+          <time>1</time>
+          <namespace>${prefix}/sc_port_base</namespace>
+          <enabled>true</enabled>
+        </plugin>
       </include>
     </gazebo>
